File: Schematics/Sensor_Board.sch (KiCad schematic (older format))
At the start: 1 part

Commit message: Added more to the schematics, basic PIC setup and CAN Transiever
Parts:
- added C? (x4): 0.1uF, symbol C
- added C?: 10uF, symbol C
- added JP?: JUMPER, symbol JUMPER
- added P?: CONN_6, symbol CONN_6
- added R?: 470, symbol R
- added R?: 10k, symbol R
- added R?: 120, symbol R
- added SW?: SW_PUSH, symbol SW_PUSH
- added U?: MCP2551SN, microchip_can-SO-08, symbol MCP2551SN
- U?: value DSPIC33E128MC506 -> DSPIC33ExxxMC50x-64TQFP
Connections:
- net labels added: +3.3V, CAN_H, CAN_L, CAN_RX, CAN_TX, GND, MCLR, PDEC2, PDED2, PGEC2, PGED2, VCC, VSS
- wire segments 0 -> 55
- no-connect marks 0 -> 1
Other:
- note added: "Note: The 2551 is a 5V standard part. \nCheck input voltage!"

Commit message: Added ADC and TI CAN Trans.
Parts:
- removed C?: 10uF, symbol C
- removed U?: MCP2551SN, microchip_can-SO-08, symbol MCP2551SN
- added 10uF: CP, symbol CP
- added C?: 0.1uF, symbol C
- added U?: SN65HVD232, symbol SN65HVD232
- added U?: AD7192, MODULE, symbol AD7192
Connections:
- net labels added: ADSCLK, AGND, AIN1, AIN2, AIN3, AIN4, AREF, BPDSW, MISO, MOSI
- wire segments 55 -> 92
- no-connect marks 1 -> 2
Other:
- moved on the sheet: C?, P?, R?, SW?

Commit message: Adding schematic with changes from yesterday
Parts:
- added 10uF, 1uF (x2): CSMALL, symbol CSMALL
- added U?: AS1359, MODULE, symbol AS1359
Connections:
- net labels added: SHD, SS, VAA
- net labels removed: VCC
- wire segments 92 -> 100
Other:
- note added: "ADC PWR"
- note added: "Need to attach output pins for ADC input pins."
- note removed: "Note: The 2551 is a 5V standard part. \nCheck input voltage!"

Commit message: Changed the ADC from AD7192 to AD7193
Parts:
- removed U?: AD7192, MODULE, symbol AD7192
- added U?: AD7193, MODULE, symbol AD7193
- U?: value AS1359 -> AS1359-3
Connections:
- net labels added: AIN5, AIN6, AIN7, AIN8, MCLK2, P2, P3, REFIN+, REFIN1-, REFIN2+, REFIN2-
- wire segments 100 -> 112

Commit message: Adding the changes from today, mainly changing some parts and basic wiring.... didn't get as much done as I would have liked
Connections:
- wire segments 112 -> 113
Other:
- moved on the sheet: C?, JP?, R?, SW?, U?

Commit message: Revert "Adding the changes from today, mainly changing some parts and basic wiring.... didn't get as much done as I would have liked"
This reverts commit 15443ba5e97c99da6254b6d753ebc1158bf0ebd2.
Connections:
- wire segments 113 -> 112
Other:
- moved on the sheet: C?, JP?, R?, SW?, U?

Commit message: Added a connector for the CAN network and some general purpose LEDs
Parts:
- added D? (x4): LED, symbol LED
- added K?: CONN_3, symbol CONN_3
- added P?: CONN_2, symbol CONN_2
Connections:
- net labels added: 3V3, LED1, LED2, LED3, LED4, RA0, RA1, RA11, RA12, RA7, RB1, RB14, RB15, RB2, RB3, RC0, RC1, RG6, RG7, RG8, RG9
- wire segments 112 -> 174
Other:
- note added: "GREEN"
- note added: "RED"
- note added: "YELLOW"
- moved on the sheet: C?, JP?, P?, R?, SW?, U?

Commit message: Added Data sheets fro the FDFMA3N109 and AP7363 chips. Plus rolling updates to schematic.
Parts:
- added C? (x2): 10uF, symbol C
- added D?: DIODE, symbol DIODE
- added P?: CONN_2, symbol CONN_2
- added P?: CONN_7X2, symbol CONN_7X2
- added R?: 38.3k, symbol R
- added R?: 8.06k, symbol R
- added U?: AP7363, MODULE, symbol AP7363
Connections:
- net labels added: RA10, RA8, RB10, RB11, RB12, RB13, RB4, RB7, RB8, RB9, RC10, RC11, RC12, RC15, RC2, RC4, RC5, RC9, RE12, RE13, RE14, RE15, REFIN1+, RF0, RF1, VBAT, Vin
- net labels removed: 3V3
- wire segments 174 -> 231
Other:
- note added: "1%"
- note added: "PMEG3050BEP\n"
- note added: "R1"
- note added: "R2"
- moved on the sheet: JP?, R?
