File: Schematics/Sensor_Board.sch (KiCad schematic (older format))
At the start: 33 parts

Commit message: Added a power switcher and an IMU, still need a compass
Parts:
- removed D?: DIODE, symbol DIODE
- added C?: 0.1uF, symbol C
- added R? (x2): 330, symbol R
- added R?: 154k, symbol R
- added R?: 10k, symbol R
- added R? (x2): 4.7k, symbol R
- added U: 1uF, symbol CSMALL
- added U (x2): 0.1uF, symbol CSMALL
- added U?: TPS2113A, MODULE, symbol TPS2113A
- added U?: MPU-6000/MPU-6050, MODULE, symbol MPU-6000/MPU-6050
- added U?: 2.2nF, symbol CSMALL
- U: renamed from 1uF; value CSMALL -> 1uF
- U: renamed from 10uF; value CSMALL -> 10uF
Connections:
- net labels added: INT_IMU, SCA_IMU, SCL_IMU, SCL_MAG, SDA_IMU, SWSTAT, V3V, VLDO
- net labels removed: RC4, RC5, RC9, RF0
- wire segments 231 -> 281
- no-connect marks 2 -> 12
Other:
- note removed: "PMEG3050BEP\n"
- moved on the sheet: 10uF, C?, R?

Commit message: Switched the IMU from MPU-6000 to MPU-9150 w/ integrated compass
Parts:
- removed U?: MPU-6000/MPU-6050, MODULE, symbol MPU-6000/MPU-6050
- added U?: MPU-9150, MODULE, symbol MPU-9150
Connections:
- no-connect marks 12 -> 13

Commit message: Added the MPU-9150 and an RGB LED to the board. Also added current limiting resistors to the status LEDs
Parts:
- added R? (x4): 330, symbol R
- added U?: 0.1uF, symbol CSMALL
- added U?: RGB_LED, MODULE, symbol RGB_LED
Connections:
- net labels added: 3V3, ES_CA, ES_CL
- net labels removed: SCL_MAG, V3V, VSS
- wire segments 281 -> 300
- no-connect marks 13 -> 10
Other:
- note added: "Analog Sensors and Power"
- note added: "CAN Transiever + Connector"
- note added: "Digital Power Flags"
- note removed: "ADC PWR"
- note removed: "Need to attach output pins for ADC input pins."
- moved on the sheet: JP?, R?, U?

Commit message: Went back to the MPU-6000 IMU based on the 9150 having a lot of issues. Also added an RGB LED for status.
Parts:
- removed U?: MPU-9150, MODULE, symbol MPU-9150
- removed U?: 0.1uF, symbol CSMALL
- added R?: 150, symbol R
- added R? (x2): 30, symbol R
- added U?: MPU-6000/MPU-6050, MODULE, symbol MPU-6000/MPU-6050
- gave numbers to parts that had none: 42
- renumbered 10uF to 10uF1, U to U11, U to U14, U to U15, U to U16, U to U3, U to U7
Connections:
- net labels added: B_LED, G_LED, IMU_CS, R_LED
- net labels removed: RA7, RG6, RG7, RG8
- wire segments 300 -> 272
Other:
- note added: "MCLR+SW &\nPICKit3 CONN"
- note added: "Status LEDs"
- note added: "Vin and Back-up Battery"
- moved on the sheet: C1, C2, C3, C4, P1, R1, R10, R11, R12, R2, R3, R4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

Commit message: started placing the pinheaders for an XBee wifi module. Also placing two nMOSFET for LED switching.
Parts:
- added P?: CONN_9X2, symbol CONN_9X2
- added P? (x2): CONN_10, symbol CONN_10
- added R19, R20: 4.7k, symbol R
- added U17, U18, U19, U21: 100uF, symbol CSMALL
- added U20: MAG3110, MODULE, symbol MAG3110
- added U8: 0.1uF, symbol CSMALL
- added U9: 1uF, symbol CSMALL
- added U?: SI1970DH, MODULE, symbol SI1970DH
- gave numbers to parts that had none: 4
Connections:
- net labels added: ES_DA, NFET_1, NFET_2, XBEE_CLK, XBEE_MISO, XBEE_MOSI, XBEE_nATTN, XBEE_nSSEL, nRESET
- net labels removed: ES_CA, RC0, RC1, RC11, RC2, RE14, RE15, SCA_IMU
- wire segments 272 -> 328
- no-connect marks 10 -> 24
Other:
- note added: "IMU + Magnetormeter"
- moved on the sheet: R14, R15

Commit message: Have to go to a meeting....
Parts:
- removed R8: 330, symbol R
- added C?: 1mF, symbol CPSMALL
- added D? (x2): LED, symbol LED
- added P?: CONN_9X2, symbol CONN_9X2
- added P? (x2): CONN_2, symbol CONN_2
- added R?: 110, symbol R
- added R?: 82, symbol R
- added R?: 50, symbol R
- added R? (x2): 4.7k, symbol R
- added U? (x4): 0.1uF, symbol CSMALL
- R10, R9: value 330 -> 110
- R12: value 330 -> 180
- R6: value 38.3k -> 36.5k
- U17, U18, U21: value 100uF -> 100nF
- U19: value 100uF -> 100n.F
Connections:
- net labels added: PWR_SW1, PWR_SW2, RC0, RC1, RC11, RC2, SLEEP_RQ
- net labels removed: RC12, RC15
- wire segments 328 -> 384
- no-connect marks 24 -> 22
Other:
- note added: "BLUE"
- note added: "XBee Wifi Pin Header"
- moved on the sheet: C5, C6, C7

Commit message: Finished the lab meeting
Parts:
- removed P?: CONN_9X2, symbol CONN_9X2
- added P?: CONN_10X2, symbol CONN_10X2
Connections:
- wire segments 384 -> 390
Other:
- moved on the sheet: C5

Commit message: Final schematic design as of 16/7/13
Parts:
- removed P?: CONN_10X2, symbol CONN_10X2
- removed R?: 82, symbol R
- added P?: CONN_9X2, symbol CONN_9X2
- added P?: CONN_2, symbol CONN_2
- added R?: 30, symbol R
Connections:
- net labels added: AN11, AN6, AN7, AN8
- net labels removed: RC0, RC1, RC11, RC2
- wire segments 390 -> 431
Other:
- note added: "Pin Out Connectors"
- note added: "uC Controlled Power Switches"
