File: Schematics/Sensor_Board.sch (KiCad schematic (older format))
At the start: 59 parts, among them P1 CONN_6, P10 CONN_10, P11 CONN_2, P12 CONN_2, P13 CONN_1, P2 CONN_2, P3 CONN_2, P5 CONN_3, P6 CONN_9X2, P7 CONN_9X2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

Commit message: Finally finished layout the board. Added the XBEE Wifi datasheet as well.
Parts:
- gave numbers to parts that had none: 1
Connections:
- net labels added: RA7, V_MAG
- net labels removed: IMU_CS
- wire segments 303 -> 304
Changed lines of the file:
@@
 Text Label 1150 6950 2    60   ~ 0
 XBEE_CLK
-Text Label 2000 6850 0    60   ~ 0
-XBEE_nSSEL
 Text Label 1150 6850 2    60   ~ 0
 XBEE_MISO
@@
 Text Label 3950 3550 0    60   ~ 0
 RB14
-Text Label 3950 3450 0    60   ~ 0
-IMU_CS
 Text Label 5000 1700 0    60   ~ 0
 CAN_L
@@
 Text Label 3850 2250 0    60   ~ 0
 B_LED
-$Comp
-L MPU-6000/MPU-6050 U22
-U 1 1 51E35339
-P 10100 5650
-F 0 "U22" H 10100 5550 50  0000 C CNN
-F 1 "MPU-6000" H 10100 5750 50  0000 C CNN
-F 2 "QFN-24" H 10100 5650 50  0001 C CNN
-F 3 "DOCUMENTATION" H 10100 5650 50  0001 C CNN
-F 4 "10.72" H 10100 5650 60  0001 C CNN "Price"
-F 5 "Digikey" H 10100 5650 60  0001 C CNN "Retailer"
-F 6 "1428-1005-1-ND" H 10100 5650 60  0001 C CNN "Part_Number"
-	1    10100 5650
-	1    0    0    -1
-$EndComp
-Text Label 9950 6450 3    60   ~ 0
-IMU_CS
 Text Notes 3000 600  0    60   ~ 0
 Status LEDs
@@
 	3800 2250 4050 2250
 Wire Wire Line
-	9950 6400 9950 6600
-Wire Wire Line
 	10050 6800 10050 6400
 Wire Wire Line
@@
 V24
 $Comp
-L CONN_3 P?
+L CONN_3 P8
 U 1 1 51F2D431
 P 1550 7600
-F 0 "P?" V 1500 7600 50  0000 C CNN
+F 0 "P8" V 1500 7600 50  0000 C CNN
 F 1 "CONN_3" V 1600 7600 40  0000 C CNN
 F 2 "PIN_ARRAY_3X1" H 1550 7600 60  0001 C CNN
@@
 Text Label 1950 7700 0    60   ~ 0
 PWR_SW3
+Text Label 7500 6250 2    60   ~ 0
+V_MAG
+Text Label 8650 6350 0    60   ~ 0
+V_MAG
+$Comp
+L MPU-6000/MPU-6050 U22
+U 1 1 51E35339
+P 10100 5650
+F 0 "U22" H 10100 5550 50  0000 C CNN
+F 1 "MPU-6000" H 10100 5750 50  0000 C CNN
+F 2 "QFN-24" H 10100 5650 50  0001 C CNN
+F 3 "DOCUMENTATION" H 10100 5650 50  0001 C CNN
+F 4 "10.72" H 10100 5650 60  0001 C CNN "Price"
+F 5 "Digikey" H 10100 5650 60  0001 C CNN "Retailer"
+F 6 "1428-1005-1-ND" H 10100 5650 60  0001 C CNN "Part_Number"
+	1    10100 5650
+	1    0    0    -1
+$EndComp
+Wire Wire Line
+	9950 6400 9950 6850
+$Comp
+L +3.3V #PWR060
+U 1 1 51F59236
+P 9800 6850
+F 0 "#PWR060" H 9800 6810 30  0001 C CNN
+F 1 "+3.3V" H 9800 6960 30  0000 C CNN
+F 2 "" H 9800 6850 60  0001 C CNN
+F 3 "" H 9800 6850 60  0001 C CNN
+	1    9800 6850
+	1    0    0    -1
+$EndComp
+Wire Wire Line
+	9950 6850 9800 6850
+Text Label 3950 3450 0    60   ~ 0
+RA7
+Text Label 2000 6850 0    60   ~ 0
+RA7
 $EndSCHEMATC

Commit message: Fixed the XBee pinheader issue. Added information onto the Silkscreen
Still Need To:
-Label Connectors
-Move Power connectors
Parts:
- removed SW1: SW_PUSH, ASL-B3F-1020, symbol SW_PUSH
- added SW1: SW_PUSH_4, symbol SW_PUSH_4
Connections:
- wire segments 304 -> 308
Changed lines of the file:
@@
 LIBS:con-commcon
 LIBS:pinhead
+LIBS:sw_push_4
 LIBS:Sensor_Board-cache
 EELAYER 24 0
@@
 PGED2
 $Comp
-L SW_PUSH SW1
-U 1 1 51D90B88
-P 900 1250
-F 0 "SW1" H 1050 1360 50  0000 C CNN
-F 1 "SW_PUSH" H 900 1170 50  0000 C CNN
-F 2 "ASL-B3F-1020" H 900 1250 60  0001 C CNN
-F 3 "" H 900 1250 60  0001 C CNN
-F 4 "0.393" H 900 1250 60  0001 C CNN "Price"
-F 5 "Digikey" H 900 1250 60  0001 C CNN "Retailer"
-F 6 "SW402-ND" H 900 1250 60  0001 C CNN "Part_Number"
-	1    900  1250
-	1    0    0    -1
-$EndComp
-$Comp
 L GND #PWR039
 U 1 1 51D90BA6
@@
 Text Label 2000 6850 0    60   ~ 0
 RA7
+$Comp
+L SW_PUSH_4 SW1
+U 1 1 51F9A416
+P 900 1250
+F 0 "SW1" H 1050 1360 50  0000 C CNN
+F 1 "SW_PUSH_4" H 900 1050 50  0000 C CNN
+F 2 "" H 900 1250 60  0000 C CNN
+F 3 "" H 900 1250 60  0000 C CNN
+	1    900  1250
+	1    0    0    -1
+$EndComp
+Wire Wire Line
+	600  1250 600  1400
+Wire Wire Line
+	600  1400 850  1400
+Wire Wire Line
+	950  1400 1200 1400
+Wire Wire Line
+	1200 1400 1200 1250
 $EndSCHEMATC

Commit message: Found out that there are two different remappable pins of the dsPIC33E. Some are input/out remappable and some are input only remappable. Fixed the XBee SPI, XBEE nRESET, and Green LED on the RGB LED to make sure they are all outputs.
Parts:
- U5: footprint 8-SOIC -> (none); Part_Number 296-26344-1-ND -> (none); Price 2.01 -> (none); Retailer Digikey -> (none)
Connections:
- net labels added: RC10, RG7
- net labels removed: RA0, RB7
Changed lines of the file:
@@
 LIBS:contrib
 LIBS:valves
+LIBS:TPS2113A
 LIBS:sn65hvd232
+LIBS:Si1970DH
+LIBS:RGB_LED
+LIBS:RESISTOR_ARRAY
+LIBS:pinhead
+LIBS:MPU-9150
+LIBS:MPU-6000_MPU-6050
+LIBS:microchip_can
+LIBS:MAG3110
+LIBS:DSPIC33E128MC506
+LIBS:dp_devices
+LIBS:AS1359
+LIBS:AP7363
+LIBS:AD7193
 LIBS:AD7192
-LIBS:AS1359
-LIBS:AD7193
-LIBS:DSPIC33E128MC506
-LIBS:AP7363
-LIBS:MPU-6000_MPU-6050
-LIBS:TPS2113A
-LIBS:MPU-9150
-LIBS:RGB_LED
-LIBS:Si1970DH
-LIBS:MAG3110
-LIBS:RESISTOR_ARRAY
-LIBS:con-commcon
-LIBS:pinhead
 LIBS:sw_push_4
 LIBS:Sensor_Board-cache
@@
 XBEE_MISO
 Text Label 2000 6750 0    60   ~ 0
-RB7
+RC10
 Text Label 1150 6750 2    60   ~ 0
 XBEE_MOSI
@@
 Text Label 7350 3450 0    60   ~ 0
 XBEE_MISO
+Text Label 7350 3750 0    60   ~ 0
+RC10
 Text Label 7350 3650 0    60   ~ 0
-RB7
-Text Label 7350 3750 0    60   ~ 0
 XBEE_MOSI
 Text Label 7350 4250 0    60   ~ 0
@@
 Text Label 6400 5650 1    60   ~ 0
 RA8
-Text Label 6300 5500 3    60   ~ 0
+Text Label 6100 5450 3    60   ~ 0
 nRESET
 Text Label 6200 5450 3    60   ~ 0
 XBEE_nATTN
-Text Label 6100 5650 1    60   ~ 0
+Text Label 6300 5650 1    60   ~ 0
 RE13
 Text Label 6000 5650 1    60   ~ 0
@@
 Text Label 3950 4750 0    60   ~ 0
 RA1
-Text Label 3950 4650 0    60   ~ 0
-RA0
+Text Label 3950 3850 0    60   ~ 0
+RG7
 Text Label 3950 4550 0    60   ~ 0
 RA11
@@
 Text Label 3950 3950 0    60   ~ 0
 B_LED
-Text Label 3950 3850 0    60   ~ 0
+Text Label 3950 4650 0    60   ~ 0
 G_LED
 Text Label 3950 3750 0    60   ~ 0
@@
 CAN_RX
 $Comp
-L SN65HVD232 U5
-U 1 1 51DA2902
-P 5600 1150
-F 0 "U5" H 5600 1400 60  0000 C CNN
-F 1 "SN65HVD232" H 5600 850 60  0000 C CNN
-F 2 "8-SOIC" H 5600 1150 60  0001 C CNN
-F 3 "" H 5600 1150 60  0001 C CNN
-F 4 "2.01" H 5600 1150 60  0001 C CNN "Price"
-F 5 "Digikey" H 5600 1150 60  0001 C CNN "Retailer"
-F 6 "296-26344-1-ND" H 5600 1150 60  0001 C CNN "Part_Number"
-	1    5600 1150
-	1    0    0    -1
-$EndComp
-$Comp
 L +3.3V #PWR047
 U 1 1 51DA29F2
@@
 RA11
 Text Label 2000 5650 0    60   ~ 0
-RA0
+RG7
 Text Label 950  5750 0    60   ~ 0
 RA1
@@
 Text Label 2000 6850 0    60   ~ 0
 RA7
+Wire Wire Line
+	600  1250 600  1400
+Wire Wire Line
+	600  1400 850  1400
+Wire Wire Line
+	950  1400 1200 1400
+Wire Wire Line
+	1200 1400 1200 1250
 $Comp
 L SW_PUSH_4 SW1
-U 1 1 51F9A416
+U 1 1 51FB057B
 P 900 1250
 F 0 "SW1" H 1050 1360 50  0000 C CNN
-F 1 "SW_PUSH_4" H 900 1050 50  0000 C CNN
+F 1 "SW_PUSH_4" H 900 1025 50  0000 C CNN
 F 2 "" H 900 1250 60  0000 C CNN
 F 3 "" H 900 1250 60  0000 C CNN
@@
 	1    0    0    -1
 $EndComp
-Wire Wire Line
-	600  1250 600  1400
-Wire Wire Line
-	600  1400 850  1400
-Wire Wire Line
-	950  1400 1200 1400
-Wire Wire Line
-	1200 1400 1200 1250
+$Comp
+L SN65HVD232 U5
+U 1 1 51FB15F1
+P 5600 1150
+F 0 "U5" H 5600 1400 60  0000 C CNN
+F 1 "SN65HVD232" H 5600 850 60  0000 C CNN
+F 2 "" H 5600 1150 60  0000 C CNN
+F 3 "" H 5600 1150 60  0000 C CNN
+	1    5600 1150
+	1    0    0    -1
+$EndComp
 $EndSCHEMATC

Commit message: Fixed the issue of pins 19 and 20 being flipped.
Connections:
- wire segments 308 -> 309
Changed lines of the file:
@@
 L GND #PWR046
 U 1 1 51DA20CD
-P 5050 6500
-F 0 "#PWR046" H 5050 6500 30  0001 C CNN
-F 1 "GND" H 5050 6430 30  0001 C CNN
-F 2 "" H 5050 6500 60  0001 C CNN
-F 3 "" H 5050 6500 60  0001 C CNN
-	1    5050 6500
+P 5550 6500
+F 0 "#PWR046" H 5550 6500 30  0001 C CNN
+F 1 "GND" H 5550 6430 30  0001 C CNN
+F 2 "" H 5550 6500 60  0001 C CNN
+F 3 "" H 5550 6500 60  0001 C CNN
+	1    5550 6500
 	1    0    0    -1
 $EndComp
@@
 L +3.3V #PWR049
 U 1 1 51E080BB
-P 5550 6400
-F 0 "#PWR049" H 5550 6360 30  0001 C CNN
-F 1 "+3.3V" H 5550 6510 30  0000 C CNN
-F 2 "" H 5550 6400 60  0001 C CNN
-F 3 "" H 5550 6400 60  0001 C CNN
-	1    5550 6400
+P 4900 6400
+F 0 "#PWR049" H 4900 6360 30  0001 C CNN
+F 1 "+3.3V" H 4900 6510 30  0000 C CNN
+F 2 "" H 4900 6400 60  0001 C CNN
+F 3 "" H 4900 6400 60  0001 C CNN
+	1    4900 6400
 	1    0    0    -1
 $EndComp
@@
 Connection ~ 5050 6400
 Wire Wire Line
-	5050 6250 5050 6500
-Wire Wire Line
 	5200 6250 5050 6250
 Wire Wire Line
@@
 	10050 4050 9750 4050
 Wire Wire Line
-	5150 6400 5050 6400
+	4900 6400 5150 6400
 Wire Wire Line
 	5750 6400 5650 6400
@@
 	1    0    0    -1
 $EndComp
+Wire Wire Line
+	5550 6400 5550 6500
+Wire Wire Line
+	5050 6400 5050 6250
 $EndSCHEMATC

Commit message: Updated to version 1.2
Connections:
- wire segments 309 -> 311
- no-connect marks 25 -> 24
Other:
- note added: "Add A 1uF cap between pin 1 and GND\nMaybe..."

Commit message: Added notes to be completed on next revision
Other:
- note added: "Add A 6.8pF and a 1uF cap between pin 1 and GND\nMaybe..."
- note added: "Add a 1k resistor to XBEE VCC\n\nAdd UART support"
- note added: "Add a speaker..... -.-\n"
- note removed: "Add A 1uF cap between pin 1 and GND\nMaybe..."
Changed lines of the file:
@@
 	7900 4400 7900 4500
 Text Notes 3200 6050 0    60   ~ 0
-Add A 1uF cap between pin 1 and GND\nMaybe...
+Add A 6.8pF and a 1uF cap between pin 1 and GND\nMaybe...
+Text Notes 8250 2500 0    60   ~ 0
+Add a speaker..... -.-\n
+Text Notes 3250 5650 0    60   ~ 0
+Add a 1k resistor to XBEE VCC\n\nAdd UART support
 $EndSCHEMATC

Commit message: Started making changes to the Sensor Board for v.2
Parts:
- removed P13: CONN_1, pinhead-1X01, symbol CONN_1
- removed P2, P3: CONN_2, PIN_ARRAY_2X1, symbol CONN_2
- removed P8: CONN_3, PIN_ARRAY_3X1, symbol CONN_3
- removed R23: 4.7k, SM0805, symbol R
- added J?: MICROCLASP_HDRX2, symbol MICROCLASP_HDRX2
- added P? (x3): CONN_1, pinhead-1X01, symbol CONN_1
- added R?: 0.2, SM0805, symbol R
- added R? (x6): 1k, SM0805, symbol R
Connections:
- net labels added: XBEE_NFET, XBEE_PWR, XBEE_RX, XBEE_TX
- net labels removed: 3V3, PWR_SW3, RA10, RB10, RB11, V24
- wire segments 311 -> 304
Other:
- note removed: "Add a 1k resistor to XBEE VCC\n\nAdd UART support"
- note removed: "Add a speaker..... -.-\n"

Commit message: Continuing changes for v2
Parts:
- added JP? (x2): PINHD-2X23, pinhead-2X23, symbol PINHD-2X23
Connections:
- wire segments 304 -> 333
Changed lines of the file:
@@
 LIBS:microclasp_hdrx2
 LIBS:microclasp_hdrx3
+LIBS:pinhd-2x23
 LIBS:Sensor_Board-cache
 EELAYER 27 0
@@
 	5750 6400 5650 6400
 Wire Wire Line
-	4900 6400 5150 6400
+	4900 6400 5050 6400
+Wire Wire Line
+	5050 6400 5150 6400
 Wire Wire Line
 	9500 4050 10050 4050
@@
 Connection ~ 5900 6150
 Wire Wire Line
-	5900 5850 5900 6200
+	5900 5850 5900 5950
+Wire Wire Line
+	5900 5950 5900 6050
+Wire Wire Line
+	5900 6050 5900 6150
+Wire Wire Line
+	5900 6150 5900 6200
 Wire Wire Line
 	6050 6400 6050 5750
@@
 	9000 6950 9000 7050
 Wire Wire Line
-	8600 7150 9450 7150
+	8600 7150 9150 7150
+Wire Wire Line
+	9150 7150 9450 7150
 Connection ~ 9150 6350
 Wire Wire Line
@@
 Connection ~ 6950 6500
 Wire Wire Line
-	6850 6500 7250 6500
+	6850 6500 6950 6500
+Wire Wire Line
+	6950 6500 7150 6500
+Wire Wire Line
+	7150 6500 7250 6500
 Wire Wire Line
 	7350 6500 7350 6450
@@
 	8650 6450 8600 6450
 Wire Wire Line
-	8600 6350 9350 6350
+	8600 6350 8750 6350
+Wire Wire Line
+	8750 6350 9000 6350
+Wire Wire Line
+	9000 6350 9150 6350
+Wire Wire Line
+	9150 6350 9350 6350
 Connection ~ 8150 5100
 Wire Wire Line
@@
 	8250 5100 8250 4500
 Wire Wire Line
-	8000 5100 8250 5100
+	8000 5100 8150 5100
+Wire Wire Line
+	8150 5100 8250 5100
 Wire Wire Line
 	8000 5100 8000 4550
@@
 Connection ~ 10150 6800
 Wire Wire Line
-	10050 6800 10250 6800
+	10050 6800 10150 6800
+Wire Wire Line
+	10150 6800 10250 6800
 Wire Wire Line
 	10250 6800 10250 6400
@@
 	9850 4900 9850 4650
 Wire Wire Line
-	10900 5900 11150 5900
+	10900 5900 11050 5900
+Wire Wire Line
+	11050 5900 11150 5900
 Wire Wire Line
 	11050 6100 11050 6150
@@
 	10150 6400 10150 6600
 Wire Wire Line
-	6300 1800 6750 1800
+	6300 1800 6450 1800
+Wire Wire Line
+	6450 1800 6750 1800
 Wire Wire Line
 	1850 3250 1150 3250
@@
 	7300 4050 7650 4050
 Wire Wire Line
-	4000 750  4000 1750
+	4000 750  4000 1050
+Wire Wire Line
+	4000 1050 4000 1350
+Wire Wire Line
+	4000 1350 4000 1650
+Wire Wire Line
+	4000 1650 4000 1750
 Wire Wire Line
 	2900 750  2650 750
@@
 	7300 3950 7650 3950
 Wire Wire Line
-	1300 1150 1300 1350
-Wire Wire Line
-	1200 1250 1400 1250
+	1300 1150 1300 1250
+Wire Wire Line
+	1300 1250 1300 1350
+Wire Wire Line
+	1200 1250 1300 1250
+Wire Wire Line
+	1300 1250 1400 1250
 Connection ~ 1300 1250
 Wire Wire Line
@@
 	7650 4150 7650 4100
 Wire Wire Line
-	7650 4100 8350 4100
+	7650 4100 7900 4100
+Wire Wire Line
+	7900 4100 8350 4100
 Wire Wire Line
 	7300 4450 7650 4450
@@
 	7650 4450 7650 4500
 Wire Wire Line
-	7650 4500 8000 4500
+	7650 4500 7900 4500
+Wire Wire Line
+	7900 4500 8000 4500
 Wire Wire Line
 	5800 2950 5800 2500
 Wire Wire Line
-	3400 4200 3700 4200
+	3400 4200 3600 4200
+Wire Wire Line
+	3600 4200 3700 4200
 Wire Wire Line
 	3700 4200 3700 4250
 Wire Wire Line
-	3250 4400 3700 4400
+	3250 4400 3600 4400
+Wire Wire Line
+	3600 4400 3700 4400
 Wire Wire Line
 	3700 4400 3700 4350
@@
 	5000 2950 5000 2650
 Wire Wire Line
-	6300 600  6750 600
+	6300 600  6450 600
+Wire Wire Line
+	6450 600  6750 600
 Wire Wire Line
 	10150 6850 10150 6800
@@
 	7950 4650 7950 5150
 Wire Wire Line
-	7950 5150 8500 5150
+	7950 5150 8350 5150
+Wire Wire Line
+	8350 5150 8500 5150
 Wire Wire Line
 	8500 5150 8500 4650
@@
 	1150 5450 900  5450
 Wire Wire Line
-	8650 7050 9450 7050
+	8650 7050 9000 7050
+Wire Wire Line
+	9000 7050 9450 7050
 Wire Notes Line
 	3050 5000 3050 3650
@@
 	6000 6300 5650 6300
 Wire Wire Line
-	5650 6300 5650 6500
+	5650 6300 5650 6400
+Wire Wire Line
+	5650 6400 5650 6500
 Wire Wire Line
 	5900 6050 5700 6050
@@
 	9500 3950 10050 3950
 Wire Wire Line
-	5350 6400 5550 6400
+	5350 6400 5450 6400
+Wire Wire Line
+	5450 6400 5550 6400
 Connection ~ 5450 6400
 Wire Wire Line
-	5950 6400 6150 6400
+	5950 6400 6050 6400
+Wire Wire Line
+	6050 6400 6150 6400
 Connection ~ 6050 6400
 Wire Wire Line
@@
 F5 "Vin" I R 2800 3250 60
 $EndSheet
+$Comp
+L PINHD-2X23 JP?
+U 1 1 52C35A2A
+P 8850 1950
+F 0 "JP?" H 8600 3175 50  0000 L BNN
+F 1 "PINHD-2X23" H 8600 550 50  0000 L BNN
+F 2 "pinhead-2X23" H 8850 2100 50  0001 C CNN
+F 3 "~" H 8850 1950 60  0000 C CNN
+	1    8850 1950
+	1    0    0    -1
+$EndComp
+$Comp
+L PINHD-2X23 JP?
+U 1 1 52C35ABE
+P 10300 1950
+F 0 "JP?" H 10050 3175 50  0000 L BNN
+F 1 "PINHD-2X23" H 10050 550 50  0000 L BNN
+F 2 "pinhead-2X23" H 10300 2100 50  0001 C CNN
+F 3 "~" H 10300 1950 60  0000 C CNN
+	1    10300 1950
+	1    0    0    -1
+$EndComp
 $EndSCHEMATC
