File: Schematics/Analog.sch (KiCad schematic (older format))
At the start: 27 parts, among them P4 CONN_7X2, U3 RESISTOR_ARRAY, U7 AD7193, U8 AS1359-3

Commit message: Put some more information for purchasing.
Parts:
- C20, C26, C27, C28, C29, C30, C34, C35, C36, C37, C38, C39: footprint (none) -> 0805
- C31: footprint (none) -> 0805; Part_Number (none) -> 311-1358-1-ND; Price (none) -> 0.059; Retailer (none) -> Digikey
- C32: Part_Number (none) -> 311-1355-1-ND; Retailer (none) -> Digikey
- P4: Part_Number (none) -> S7075-ND; Price (none) -> 0.959; Retailer (none) -> Digikey
Changed lines of the file:
@@
-EESchema Schematic File Version 2  date Thu 18 Jul 2013 06:36:55 PM PDT
+EESchema Schematic File Version 2  date Fri 19 Jul 2013 02:27:14 PM PDT
 LIBS:power
 LIBS:device
@@
 $EndDescr
 $Comp
+L CSMALL C31
+U 1 1 51E99A6D
+P 4400 3950
+F 0 "C31" H 4400 4000 30  0000 L CNN
+F 1 "1uF" H 4400 3900 30  0000 L CNN
+F 2 "0805" H 4400 3950 60  0001 C CNN
+F 4 "0.059" H 4400 3950 60  0001 C CNN "Price"
+F 5 "Digikey" H 4400 3950 60  0001 C CNN "Retailer"
+F 6 "311-1358-1-ND" H 4400 3950 60  0001 C CNN "Part_Number"
+	1    4400 3950
+	1    0    0    -1
+$EndComp
+$Comp
+L CSMALL C32
+U 1 1 51E99976
+P 6400 4100
+F 0 "C32" H 6400 4050 30  0000 L CNN
+F 1 "10uF" H 6400 4150 30  0000 L CNN
+F 2 "0805" H 6400 4100 60  0001 C CNN
+F 4 "0.11" V 6400 4100 60  0001 C CNN "Price"
+F 5 "Digikey" H 6400 4100 60  0001 C CNN "Retailer"
+F 6 "311-1355-1-ND" H 6400 4100 60  0001 C CNN "Part_Number"
+	1    6400 4100
+	0    1    1    0
+$EndComp
+$Comp
+L CSMALL C34
+U 1 1 51E997A5
+P 7250 3500
+F 0 "C34" H 7275 3550 30  0000 L CNN
+F 1 "0.1uF" H 7150 3450 30  0000 L CNN
+F 2 "0805" H 7250 3500 60  0001 C CNN
+F 4 "0.01152" H 7250 3500 60  0001 C CNN "Price"
+F 5 "Digikey" H 7250 3500 60  0001 C CNN "Retailer"
+F 6 "1276-1007-1-ND" H 7250 3500 60  0001 C CNN "Part_Number"
+	1    7250 3500
+	-1   0    0    -1
+$EndComp
+$Comp
+L CSMALL C35
+U 1 1 51E997A3
+P 7350 3400
+F 0 "C35" H 7375 3450 30  0000 L CNN
+F 1 "0.1uF" H 7250 3350 30  0000 L CNN
+F 2 "0805" H 7350 3400 60  0001 C CNN
+F 4 "0.01152" H 7350 3400 60  0001 C CNN "Price"
+F 5 "Digikey" H 7350 3400 60  0001 C CNN "Retailer"
+F 6 "1276-1007-1-ND" H 7350 3400 60  0001 C CNN "Part_Number"
+	1    7350 3400
+	-1   0    0    -1
+$EndComp
+$Comp
+L CSMALL C36
+U 1 1 51E997A2
+P 7450 3300
+F 0 "C36" H 7475 3350 30  0000 L CNN
+F 1 "0.1uF" H 7350 3250 30  0000 L CNN
+F 2 "0805" H 7450 3300 60  0001 C CNN
+F 4 "0.01152" H 7450 3300 60  0001 C CNN "Price"
+F 5 "Digikey" H 7450 3300 60  0001 C CNN "Retailer"
+F 6 "1276-1007-1-ND" H 7450 3300 60  0001 C CNN "Part_Number"
+	1    7450 3300
+	-1   0    0    -1
+$EndComp
+$Comp
+L CSMALL C37
+U 1 1 51E997A1
+P 7550 3200
+F 0 "C37" H 7575 3250 30  0000 L CNN
+F 1 "0.1uF" H 7450 3150 30  0000 L CNN
+F 2 "0805" H 7550 3200 60  0001 C CNN
+F 4 "0.01152" H 7550 3200 60  0001 C CNN "Price"
+F 5 "Digikey" H 7550 3200 60  0001 C CNN "Retailer"
+F 6 "1276-1007-1-ND" H 7550 3200 60  0001 C CNN "Part_Number"
+	1    7550 3200
+	-1   0    0    -1
+$EndComp
+$Comp
+L CSMALL C38
+U 1 1 51E997A0
+P 8000 3250
+F 0 "C38" H 8025 3300 30  0000 L CNN
+F 1 "0.1uF" H 7900 3200 30  0000 L CNN
+F 2 "0805" H 8000 3250 60  0001 C CNN
+F 4 "0.01152" H 8000 3250 60  0001 C CNN "Price"
+F 5 "Digikey" H 8000 3250 60  0001 C CNN "Retailer"
+F 6 "1276-1007-1-ND" H 8000 3250 60  0001 C CNN "Part_Number"
+	1    8000 3250
+	-1   0    0    -1
+$EndComp
+$Comp
+L CSMALL C30
+U 1 1 51E9978E
+P 3850 3500
+F 0 "C30" H 3875 3550 30  0000 L CNN
+F 1 "0.1uF" H 3750 3450 30  0000 L CNN
+F 2 "0805" H 3850 3500 60  0001 C CNN
+F 4 "0.01152" H 3850 3500 60  0001 C CNN "Price"
+F 5 "Digikey" H 3850 3500 60  0001 C CNN "Retailer"
+F 6 "1276-1007-1-ND" H 3850 3500 60  0001 C CNN "Part_Number"
+	1    3850 3500
+	-1   0    0    -1
+$EndComp
+$Comp
+L CSMALL C29
+U 1 1 51E9978D
+P 3750 3400
+F 0 "C29" H 3775 3450 30  0000 L CNN
+F 1 "0.1uF" H 3650 3350 30  0000 L CNN
+F 2 "0805" H 3750 3400 60  0001 C CNN
+F 4 "0.01152" H 3750 3400 60  0001 C CNN "Price"
+F 5 "Digikey" H 3750 3400 60  0001 C CNN "Retailer"
+F 6 "1276-1007-1-ND" H 3750 3400 60  0001 C CNN "Part_Number"
+	1    3750 3400
+	-1   0    0    -1
+$EndComp
+$Comp
+L CSMALL C28
+U 1 1 51E9978C
+P 3650 3300
+F 0 "C28" H 3675 3350 30  0000 L CNN
+F 1 "0.1uF" H 3550 3250 30  0000 L CNN
+F 2 "0805" H 3650 3300 60  0001 C CNN
+F 4 "0.01152" H 3650 3300 60  0001 C CNN "Price"
+F 5 "Digikey" H 3650 3300 60  0001 C CNN "Retailer"
+F 6 "1276-1007-1-ND" H 3650 3300 60  0001 C CNN "Part_Number"
+	1    3650 3300
+	-1   0    0    -1
+$EndComp
+$Comp
+L CSMALL C27
+U 1 1 51E9978B
+P 3550 3200
+F 0 "C27" H 3575 3250 30  0000 L CNN
+F 1 "0.1uF" H 3450 3150 30  0000 L CNN
+F 2 "0805" H 3550 3200 60  0001 C CNN
+F 4 "0.01152" H 3550 3200 60  0001 C CNN "Price"
+F 5 "Digikey" H 3550 3200 60  0001 C CNN "Retailer"
+F 6 "1276-1007-1-ND" H 3550 3200 60  0001 C CNN "Part_Number"
+	1    3550 3200
+	-1   0    0    -1
+$EndComp
+$Comp
+L CSMALL C26
+U 1 1 51E9978A
+P 3250 3250
+F 0 "C26" H 3275 3300 30  0000 L CNN
+F 1 "0.1uF" H 3150 3200 30  0000 L CNN
+F 2 "0805" H 3250 3250 60  0001 C CNN
+F 4 "0.01152" H 3250 3250 60  0001 C CNN "Price"
+F 5 "Digikey" H 3250 3250 60  0001 C CNN "Retailer"
+F 6 "1276-1007-1-ND" H 3250 3250 60  0001 C CNN "Part_Number"
+	1    3250 3250
+	-1   0    0    -1
+$EndComp
+$Comp
 L CSMALL C39
 U 1 1 51E8641D
@@
 F 0 "C39" H 8225 3300 30  0000 L CNN
 F 1 "0.1uF" H 8100 3200 30  0000 L CNN
+F 2 "0805" H 8200 3250 60  0001 C CNN
 F 4 "0.01152" H 8200 3250 60  0001 C CNN "Price"
 F 5 "Digikey" H 8200 3250 60  0001 C CNN "Retailer"
 F 6 "1276-1007-1-ND" H 8200 3250 60  0001 C CNN "Part_Number"
 	1    8200 3250
-	-1   0    0    -1
-$EndComp
-$Comp
-L CSMALL C38
-U 1 1 51E8641A
-P 8000 3250
-F 0 "C38" H 8025 3300 30  0000 L CNN
-F 1 "0.1uF" H 7900 3200 30  0000 L CNN
-F 4 "0.01152" H 8000 3250 60  0001 C CNN "Price"
-F 5 "Digikey" H 8000 3250 60  0001 C CNN "Retailer"
-F 6 "1276-1007-1-ND" H 8000 3250 60  0001 C CNN "Part_Number"
-	1    8000 3250
-	-1   0    0    -1
-$EndComp
-$Comp
-L CSMALL C37
-U 1 1 51E86419
-P 7550 3200
-F 0 "C37" H 7575 3250 30  0000 L CNN
-F 1 "0.1uF" H 7450 3150 30  0000 L CNN
-F 4 "0.01152" H 7550 3200 60  0001 C CNN "Price"
-F 5 "Digikey" H 7550 3200 60  0001 C CNN "Retailer"
-F 6 "1276-1007-1-ND" H 7550 3200 60  0001 C CNN "Part_Number"
-	1    7550 3200
-	-1   0    0    -1
-$EndComp
-$Comp
-L CSMALL C36
-U 1 1 51E86418
-P 7450 3300
-F 0 "C36" H 7475 3350 30  0000 L CNN
-F 1 "0.1uF" H 7350 3250 30  0000 L CNN
-F 4 "0.01152" H 7450 3300 60  0001 C CNN "Price"
-F 5 "Digikey" H 7450 3300 60  0001 C CNN "Retailer"
-F 6 "1276-1007-1-ND" H 7450 3300 60  0001 C CNN "Part_Number"
-	1    7450 3300
-	-1   0    0    -1
-$EndComp
-$Comp
-L CSMALL C35
-U 1 1 51E86417
-P 7350 3400
-F 0 "C35" H 7375 3450 30  0000 L CNN
-F 1 "0.1uF" H 7250 3350 30  0000 L CNN
-F 4 "0.01152" H 7350 3400 60  0001 C CNN "Price"
-F 5 "Digikey" H 7350 3400 60  0001 C CNN "Retailer"
-F 6 "1276-1007-1-ND" H 7350 3400 60  0001 C CNN "Part_Number"
-	1    7350 3400
-	-1   0    0    -1
-$EndComp
-$Comp
-L CSMALL C34
-U 1 1 51E86415
-P 7250 3500
-F 0 "C34" H 7275 3550 30  0000 L CNN
-F 1 "0.1uF" H 7150 3450 30  0000 L CNN
-F 4 "0.01152" H 7250 3500 60  0001 C CNN "Price"
-F 5 "Digikey" H 7250 3500 60  0001 C CNN "Retailer"
-F 6 "1276-1007-1-ND" H 7250 3500 60  0001 C CNN "Part_Number"
-	1    7250 3500
-	-1   0    0    -1
-$EndComp
-$Comp
-L CSMALL C30
-U 1 1 51E86410
-P 3850 3500
-F 0 "C30" H 3875 3550 30  0000 L CNN
-F 1 "0.1uF" H 3750 3450 30  0000 L CNN
-F 4 "0.01152" H 3850 3500 60  0001 C CNN "Price"
-F 5 "Digikey" H 3850 3500 60  0001 C CNN "Retailer"
-F 6 "1276-1007-1-ND" H 3850 3500 60  0001 C CNN "Part_Number"
-	1    3850 3500
-	-1   0    0    -1
-$EndComp
-$Comp
-L CSMALL C29
-U 1 1 51E8640D
-P 3750 3400
-F 0 "C29" H 3775 3450 30  0000 L CNN
-F 1 "0.1uF" H 3650 3350 30  0000 L CNN
-F 4 "0.01152" H 3750 3400 60  0001 C CNN "Price"
-F 5 "Digikey" H 3750 3400 60  0001 C CNN "Retailer"
-F 6 "1276-1007-1-ND" H 3750 3400 60  0001 C CNN "Part_Number"
-	1    3750 3400
-	-1   0    0    -1
-$EndComp
-$Comp
-L CSMALL C28
-U 1 1 51E8640C
-P 3650 3300
-F 0 "C28" H 3675 3350 30  0000 L CNN
-F 1 "0.1uF" H 3550 3250 30  0000 L CNN
-F 4 "0.01152" H 3650 3300 60  0001 C CNN "Price"
-F 5 "Digikey" H 3650 3300 60  0001 C CNN "Retailer"
-F 6 "1276-1007-1-ND" H 3650 3300 60  0001 C CNN "Part_Number"
-	1    3650 3300
-	-1   0    0    -1
-$EndComp
-$Comp
-L CSMALL C27
-U 1 1 51E8640B
-P 3550 3200
-F 0 "C27" H 3575 3250 30  0000 L CNN
-F 1 "0.1uF" H 3450 3150 30  0000 L CNN
-F 4 "0.01152" H 3550 3200 60  0001 C CNN "Price"
-F 5 "Digikey" H 3550 3200 60  0001 C CNN "Retailer"
-F 6 "1276-1007-1-ND" H 3550 3200 60  0001 C CNN "Part_Number"
-	1    3550 3200
-	-1   0    0    -1
-$EndComp
-$Comp
-L CSMALL C26
-U 1 1 51E86409
-P 3250 3250
-F 0 "C26" H 3275 3300 30  0000 L CNN
-F 1 "0.1uF" H 3150 3200 30  0000 L CNN
-F 4 "0.01152" H 3250 3250 60  0001 C CNN "Price"
-F 5 "Digikey" H 3250 3250 60  0001 C CNN "Retailer"
-F 6 "1276-1007-1-ND" H 3250 3250 60  0001 C CNN "Part_Number"
-	1    3250 3250
 	-1   0    0    -1
 $EndComp
@@
 F 0 "C20" H 3075 3300 30  0000 L CNN
 F 1 "0.1uF" H 2950 3200 30  0000 L CNN
+F 2 "0805" H 3050 3250 60  0001 C CNN
 F 4 "0.01152" H 3050 3250 60  0001 C CNN "Price"
 F 5 "Digikey" H 3050 3250 60  0001 C CNN "Retailer"
@@
 $EndComp
 $Comp
-L CSMALL C32
-U 1 1 51E814BA
-P 6400 4100
-F 0 "C32" V 6350 4150 30  0000 L CNN
-F 1 "10uF" V 6450 4150 30  0000 L CNN
-F 2 "0805" H 6400 4100 60  0001 C CNN
-F 4 "0.11" V 6400 4100 60  0001 C CNN "Price"
-	1    6400 4100
-	0    -1   -1   0
-$EndComp
-$Comp
-L CSMALL C31
-U 1 1 51E814B9
-P 4400 3950
-F 0 "C31" H 4425 4000 30  0000 L CNN
-F 1 "1uF" H 4400 3900 30  0000 L CNN
-	1    4400 3950
-	1    0    0    -1
-$EndComp
-$Comp
 L VAA #PWR083
 U 1 1 51E814B8
@@
 F 0 "P4" H 6500 5450 60  0000 C CNN
 F 1 "CONN_7X2" V 6500 5050 60  0000 C CNN
+F 4 "0.959" H 6500 5050 60  0001 C CNN "Price"
+F 5 "Digikey" H 6500 5050 60  0001 C CNN "Retailer"
+F 6 "S7075-ND" H 6500 5050 60  0001 C CNN "Part_Number"
 	1    6500 5050
 	1    0    0    -1

Commit message: Made a BOM and tried to complete it as much as possible. Had to use the xml->csv method described in KiCAD's documentation.
Parts:
- C33: Part_Number (none) -> 311-1358-1-ND; Part_number 311-1358-1-ND -> (none)
Changed lines of the file:
@@
 F 4 "0.059" H 6500 4250 60  0001 C CNN "Price"
 F 5 "Digikey" H 6500 4250 60  0001 C CNN "Retailer"
-F 6 "311-1358-1-ND" H 6500 4250 60  0001 C CNN "Part_number"
+F 6 "311-1358-1-ND" H 6500 4250 60  0001 C CNN "Part_Number"
 	1    6500 4250
 	1    0    0    -1
