File: Schematics/Analog.sch (KiCad schematic (older format))
At the start: 38 parts, among them U7 AD7193, U8 AS1359-3

Commit message: Almost finished with V2.0 of the sensor board. Need to add one more trace... hopefully.
Parts:
- gave numbers to parts that had none: 13
Connections:
- net labels removed: REFIN2+, REFIN2-
- wire segments 124 -> 122
- no-connect marks 3 -> 5

Commit message: Changed the 3.3V->3V LDO from AS1359 to AS1953 Still need to work on refactoring schematic for new version of KiCAD
Parts:
- removed C32: 10nF, c_0805, symbol CSMALL
- removed C33: 1uF, c_0805, symbol CSMALL
- added C32: 0.01uF, symbol Csmall
- added C33: 1uF, symbol Csmall
- U8: value AS1359-3 -> AS1353-30; Part_Number AS1359-BTTT-30CT-ND -> AS1353-30
Connections:
- wire segments 122 -> 124
Changed lines of the file:
@@
 LIBS:dp_devices
 LIBS:DSPIC33E128MC506
+LIBS:ld29150dt50r
 LIBS:MAG3110
 LIBS:microchip_can
+LIBS:microclasp_hdrx2
+LIBS:microclasp_hdrx3
 LIBS:MPU-6000_MPU-6050
 LIBS:MPU-9150
+LIBS:ncp59151ds50r4g
+LIBS:pinhd-2x23
 LIBS:pinhead
 LIBS:RESISTOR_ARRAY
@@
 LIBS:sw_push_4
 LIBS:TPS2113A
-LIBS:microclasp_hdrx2
-LIBS:microclasp_hdrx3
-LIBS:pinhd-2x23
-LIBS:ld29150dt50r
-LIBS:ncp59151ds50r4g
-LIBS:Sensor_Board-cache
-EELAYER 27 0
+EELAYER 24 0
 EELAYER END
 $Descr A4 11693 8268
@@
 	1    4400 3950
 	1    0    0    -1
-$EndComp
-$Comp
-L CSMALL C32
-U 1 1 51E99976
-P 6400 4100
-F 0 "C32" H 6400 4050 30  0000 L CNN
-F 1 "10nF" H 6400 4150 30  0000 L CNN
-F 2 "c_0805" H 6400 4100 60  0001 C CNN
-F 3 "" H 6400 4100 60  0001 C CNN
-F 4 "0.11" V 6400 4100 60  0001 C CNN "Price"
-F 5 "Digikey" H 6400 4100 60  0001 C CNN "Retailer"
-F 6 "311-1355-1-ND" H 6400 4100 60  0001 C CNN "Part_Number"
-	1    6400 4100
-	0    1    1    0
 $EndComp
 $Comp
@@
 $EndComp
 $Comp
-L CSMALL C33
-U 1 1 51E814BB
-P 6500 4250
-F 0 "C33" H 6525 4300 30  0000 L CNN
-F 1 "1uF" H 6500 4200 30  0000 L CNN
-F 2 "c_0805" H 6500 4250 60  0001 C CNN
-F 3 "" H 6500 4250 60  0001 C CNN
-F 4 "0.059" H 6500 4250 60  0001 C CNN "Price"
-F 5 "Digikey" H 6500 4250 60  0001 C CNN "Retailer"
-F 6 "311-1358-1-ND" H 6500 4250 60  0001 C CNN "Part_Number"
-	1    6500 4250
-	1    0    0    -1
-$EndComp
-$Comp
-L VAA #PWR063
-U 1 1 51E814B8
-P 6550 4000
-F 0 "#PWR063" H 6550 4060 30  0001 C CNN
-F 1 "VAA" H 6550 4110 30  0000 C CNN
-F 2 "" H 6550 4000 60  0001 C CNN
-F 3 "" H 6550 4000 60  0001 C CNN
-	1    6550 4000
-	1    0    0    -1
-$EndComp
-$Comp
 L VAA #PWR064
 U 1 1 51E814B7
@@
 P 5600 4000
 F 0 "U8" H 5350 4200 50  0000 C CNN
-F 1 "AS1359-3" H 5600 3800 50  0000 C CNN
+F 1 "AS1353-30" H 5600 3800 50  0000 C CNN
 F 2 "dp_devices-SOT-23-5" H 5600 4000 50  0001 C CNN
 F 3 "DOCUMENTATION" H 5600 4000 50  0001 C CNN
 F 4 "1.75" H 5600 4000 60  0001 C CNN "Price"
 F 5 "Digikey" H 5600 4000 60  0001 C CNN "Retailer"
-F 6 "AS1359-BTTT-30CT-ND" H 5600 4000 60  0001 C CNN "Part_Number"
+F 6 "AS1353-30" H 5600 4000 60  0001 C CNN "Part_Number"
 	1    5600 4000
 	1    0    0    -1
@@
 L AGND #PWR069
 U 1 1 51E814AF
-P 6500 4400
-F 0 "#PWR069" H 6500 4400 40  0001 C CNN
-F 1 "AGND" H 6500 4330 50  0000 C CNN
-F 2 "" H 6500 4400 60  0001 C CNN
-F 3 "" H 6500 4400 60  0001 C CNN
-	1    6500 4400
+P 6500 4850
+F 0 "#PWR069" H 6500 4850 40  0001 C CNN
+F 1 "AGND" H 6500 4780 50  0000 C CNN
+F 2 "" H 6500 4850 60  0001 C CNN
+F 3 "" H 6500 4850 60  0001 C CNN
+	1    6500 4850
 	1    0    0    -1
 $EndComp
@@
 	1    0    0    -1
 $EndComp
-Text Label 6300 4000 0    60   ~ 0
-VAA
 NoConn ~ 4600 2200
 NoConn ~ 4600 2500
@@
 	6500 2700 7250 2700
 Wire Wire Line
-	6500 4350 6500 4400
-Connection ~ 6500 4100
-Connection ~ 6500 4000
-Wire Wire Line
-	6500 4000 6500 4150
-Wire Wire Line
-	6250 4100 6300 4100
+	6500 4350 6500 4850
 Wire Wire Line
 	4700 4050 4400 4050
@@
 Wire Wire Line
 	4400 3850 4400 3800
-Wire Wire Line
-	6250 4000 6550 4000
 Wire Wire Line
 	5350 900  5350 950
@@
 NoConn ~ 4600 2700
 NoConn ~ 4600 2800
+$Comp
+L Csmall C33
+U 1 1 53A1C920
+P 6500 4250
+F 0 "C33" H 6525 4300 30  0000 L CNN
+F 1 "1uF" H 6525 4200 30  0000 L CNN
+F 2 "" H 6500 4250 60  0000 C CNN
+F 3 "" H 6500 4250 60  0000 C CNN
+	1    6500 4250
+	1    0    0    -1
+$EndComp
+$Comp
+L Csmall C32
+U 1 1 53A1C9FE
+P 6300 4250
+F 0 "C32" H 6325 4300 30  0000 L CNN
+F 1 "0.01uF" H 6325 4200 30  0000 L CNN
+F 2 "" H 6300 4250 60  0000 C CNN
+F 3 "" H 6300 4250 60  0000 C CNN
+	1    6300 4250
+	1    0    0    -1
+$EndComp
+Wire Wire Line
+	6250 4000 6500 4000
+Wire Wire Line
+	6500 4000 6500 4150
+Wire Wire Line
+	6250 4100 6300 4100
+Wire Wire Line
+	6300 4100 6300 4150
+Wire Wire Line
+	6300 4350 6500 4350
 $EndSCHEMATC
