File: Schematics/Vin_and_BackUp.sch (KiCad schematic (older format))
At the start: 16 parts, among them U1 TPS2113A, U2 AP7363-33, U9 SI1967DH

Commit message: Changed the Voltage in so that the board will take voltage from the Motor board or supply voltage when the 24V is pulled
Parts:
- gave numbers to parts that had none: 1
Changed lines of the file:
@@
 $EndComp
 $Comp
-L GND #PWR88
+L GND #PWR082
 U 1 1 51EB0A6A
 P 6550 3500
-F 0 "#PWR88" H 6550 3500 30  0001 C CNN
+F 0 "#PWR082" H 6550 3500 30  0001 C CNN
 F 1 "GND" H 6550 3430 30  0001 C CNN
 F 2 "" H 6550 3500 60  0001 C CNN
@@
 1%
 $Comp
-L GND #PWR83
+L GND #PWR083
 U 1 1 51EB0A96
 P 4000 2000
-F 0 "#PWR83" H 4000 2000 30  0001 C CNN
+F 0 "#PWR083" H 4000 2000 30  0001 C CNN
 F 1 "GND" H 4000 1930 30  0001 C CNN
 F 2 "" H 4000 2000 60  0001 C CNN
@@
 $EndComp
 $Comp
-L GND #PWR78
+L GND #PWR084
 U 1 1 51EB0EDC
 P 3000 4350
-F 0 "#PWR78" H 3000 4350 30  0001 C CNN
+F 0 "#PWR084" H 3000 4350 30  0001 C CNN
 F 1 "GND" H 3000 4280 30  0001 C CNN
 F 2 "" H 3000 4350 60  0001 C CNN
@@
 $EndComp
 $Comp
-L GND #PWR82
+L GND #PWR085
 U 1 1 51EB0EE2
 P 3850 4800
-F 0 "#PWR82" H 3850 4800 30  0001 C CNN
+F 0 "#PWR085" H 3850 4800 30  0001 C CNN
 F 1 "GND" H 3850 4730 30  0001 C CNN
 F 2 "" H 3850 4800 60  0001 C CNN
@@
 VLDO
 $Comp
-L GND #PWR86
+L GND #PWR086
 U 1 1 51EB0EEA
 P 5350 4800
-F 0 "#PWR86" H 5350 4800 30  0001 C CNN
+F 0 "#PWR086" H 5350 4800 30  0001 C CNN
 F 1 "GND" H 5350 4730 30  0001 C CNN
 F 2 "" H 5350 4800 60  0001 C CNN
@@
 $EndComp
 $Comp
-L GND #PWR87
+L GND #PWR087
 U 1 1 51EB0EF0
 P 5700 4800
-F 0 "#PWR87" H 5700 4800 30  0001 C CNN
+F 0 "#PWR087" H 5700 4800 30  0001 C CNN
 F 1 "GND" H 5700 4730 30  0001 C CNN
 F 2 "" H 5700 4800 60  0001 C CNN
@@
 Vbatt
 $Comp
-L GND #PWR84
+L GND #PWR088
 U 1 1 51EB10FB
 P 4850 3300
-F 0 "#PWR84" H 4850 3300 30  0001 C CNN
+F 0 "#PWR088" H 4850 3300 30  0001 C CNN
 F 1 "GND" H 4850 3230 30  0001 C CNN
 F 2 "" H 4850 3300 60  0001 C CNN
@@
 $EndComp
 $Comp
-L GND #PWR81
+L GND #PWR089
 U 1 1 51EB119F
 P 3850 3800
-F 0 "#PWR81" H 3850 3800 30  0001 C CNN
+F 0 "#PWR089" H 3850 3800 30  0001 C CNN
 F 1 "GND" H 3850 3730 30  0001 C CNN
 F 2 "" H 3850 3800 60  0001 C CNN
@@
 $EndComp
 $Comp
-L GND #PWR79
+L GND #PWR090
 U 1 1 51EB11FB
 P 3550 3850
-F 0 "#PWR79" H 3550 3850 30  0001 C CNN
+F 0 "#PWR090" H 3550 3850 30  0001 C CNN
 F 1 "GND" H 3550 3780 30  0001 C CNN
 F 2 "" H 3550 3850 60  0001 C CNN
@@
 $EndComp
 $Comp
-L GND #PWR85
+L GND #PWR091
 U 1 1 51EB154E
 P 4450 2500
-F 0 "#PWR85" H 4450 2500 30  0001 C CNN
+F 0 "#PWR091" H 4450 2500 30  0001 C CNN
 F 1 "GND" H 4450 2430 30  0001 C CNN
 F 2 "" H 4450 2500 60  0001 C CNN
@@
 Vmotor
 $Comp
-L +3.3V #PWR80
+L +3.3V #PWR092
 U 1 1 51EB404B
 P 3650 1850
-F 0 "#PWR80" H 3650 1810 30  0001 C CNN
+F 0 "#PWR092" H 3650 1810 30  0001 C CNN
 F 1 "+3.3V" H 3650 1960 30  0000 C CNN
 F 2 "" H 3650 1850 60  0001 C CNN
@@
 Connection ~ 3650 2450
 $Comp
-L R R?
+L R R6
 U 1 1 51EB4833
 P 3650 2150
-F 0 "R?" V 3730 2150 40  0000 C CNN
+F 0 "R6" V 3730 2150 40  0000 C CNN
 F 1 "200" V 3657 2151 40  0000 C CNN
 F 2 "0805" H 3650 2150 60  0001 C CNN

Commit message: Made a BOM and tried to complete it as much as possible. Had to use the xml->csv method described in KiCAD's documentation.
Parts:
- C4: Field6 PCE3855CT-ND -> (none); Part_Number (none) -> PCE3855CT-ND
- R6: Part)Number RMCF0805JT200RCT-ND -> (none); Part_Number (none) -> RMCF0805JT200RCT-ND
- U1: Part_Number (none) -> 296-16938-1-ND; Part_Numver 296-16938-1-ND -> (none)
- U9: footprint MODULE -> 6-TSSOP; Part_Number (none) -> SI1967DH-T1-GE3CT-ND; Price (none) -> 0.5; Retailer (none) -> Digikey
Connections:
- wire segments 44 -> 46
Changed lines of the file:
@@
 F 4 "0.81" H 5200 3150 60  0001 C CNN "Price"
 F 5 "Digikey" H 5200 3150 60  0001 C CNN "Retailer"
-F 6 "PCE3855CT-ND" H 5200 3150 60  0001 C CNN "Field6"
+F 6 "PCE3855CT-ND" H 5200 3150 60  0001 C CNN "Part_Number"
 	1    5200 3150
 	1    0    0    -1
@@
 F 4 "2.15" H 4350 3100 60  0001 C CNN "Price"
 F 5 "Digikey" H 4350 3100 60  0001 C CNN "Retailer"
-F 6 "296-16938-1-ND" H 4350 3100 60  0001 C CNN "Part_Numver"
+F 6 "296-16938-1-ND" H 4350 3100 60  0001 C CNN "Part_Number"
 	1    4350 3100
 	1    0    0    -1
@@
 F 0 "U9" H 4500 1850 50  0000 C CNN
 F 1 "SI1967DH" H 4650 1450 50  0000 C CNN
-F 2 "MODULE" H 4650 1650 50  0001 C CNN
+F 2 "6-TSSOP" H 4650 1650 50  0001 C CNN
 F 3 "DOCUMENTATION" H 4650 1650 50  0001 C CNN
+F 4 "0.5" H 4650 1650 60  0001 C CNN "Price"
+F 5 "Digikey" H 4650 1650 60  0001 C CNN "Retailer"
+F 6 "SI1967DH-T1-GE3CT-ND" H 4650 1650 60  0001 C CNN "Part_Number"
 	1    4650 1650
 	1    0    0    -1
@@
 F 4 "0.029" V 3650 2150 60  0001 C CNN "Price"
 F 5 "Digikey" V 3650 2150 60  0001 C CNN "Retailer"
-F 6 "RMCF0805JT200RCT-ND" V 3650 2150 60  0001 C CNN "Part)Number"
+F 6 "RMCF0805JT200RCT-ND" V 3650 2150 60  0001 C CNN "Part_Number"
 	1    3650 2150
 	-1   0    0    1
@@
 Wire Wire Line
 	4350 2450 4450 2450
+$Comp
+L GND #PWR093
+U 1 1 51EC40C7
+P 5200 3350
+F 0 "#PWR093" H 5200 3350 30  0001 C CNN
+F 1 "GND" H 5200 3280 30  0001 C CNN
+F 2 "" H 5200 3350 60  0001 C CNN
+F 3 "" H 5200 3350 60  0001 C CNN
+	1    5200 3350
+	1    0    0    -1
+$EndComp
+Wire Wire Line
+	5200 3250 5200 3350
+$Comp
+L GND #PWR094
+U 1 1 51EC4101
+P 5400 3650
+F 0 "#PWR094" H 5400 3650 30  0001 C CNN
+F 1 "GND" H 5400 3580 30  0001 C CNN
+F 2 "" H 5400 3650 60  0001 C CNN
+F 3 "" H 5400 3650 60  0001 C CNN
+	1    5400 3650
+	1    0    0    -1
+$EndComp
+Wire Wire Line
+	5400 3550 5400 3650
 $EndSCHEMATC

Commit message: Associated all components with either foot prints for layout. Also added library and module files for various components.
Parts:
- removed R17: 51, 0805, symbol R
- removed U9: SI1967DH, 6-TSSOP, symbol SI1967DH
- added U9: SI1970DH, MODULE, symbol SI1970DH
- R3: value 1580 -> 200
- R5: value 330 -> 390; Part_Number RMCF0805JT330RCT-ND -> RMCF0805JT390RCT-ND
Connections:
- net labels added: V24
- net labels removed: Dmotor
- wire segments 46 -> 45
Changed lines of the file:
@@
 LIBS:MAG3110
 LIBS:RESISTOR_ARRAY
+LIBS:con-commcon
+LIBS:pinhead
 LIBS:Sensor_Board-cache
 EELAYER 24 0
@@
 L CSMALL C3
 U 1 1 51EB0A40
-P 4000 1850
-F 0 "C3" H 4000 1900 30  0000 L CNN
-F 1 "1uF" H 4000 1800 30  0000 L CNN
-F 2 "0805" H 4000 1850 60  0001 C CNN
-F 3 "" H 4000 1850 60  0001 C CNN
-F 4 "0.059" H 4000 1850 60  0001 C CNN "Price"
-F 5 "Digikey" H 4000 1850 60  0001 C CNN "Retailer"
-F 6 "311-1358-1-ND" H 4000 1850 60  0001 C CNN "Part_Number"
-	1    4000 1850
-	1    0    0    -1
-$EndComp
-$Comp
-L R R17
-U 1 1 51EB0A49
-P 5400 3300
-F 0 "R17" V 5480 3300 40  0000 C CNN
-F 1 "51" V 5407 3301 40  0000 C CNN
-F 2 "0805" H 5400 3300 60  0001 C CNN
-F 3 "" H 5400 3300 60  0001 C CNN
-F 4 "0.021" V 5400 3300 60  0001 C CNN "Price"
-F 5 "Digikey" V 5400 3300 60  0001 C CNN "Retailer"
-F 6 "RMCF0805JT51R0CT-ND" V 5400 3300 60  0001 C CNN "Part_Number"
-	1    5400 3300
-	-1   0    0    1
+P 3850 1650
+F 0 "C3" H 3850 1700 30  0000 L CNN
+F 1 "1uF" H 3850 1600 30  0000 L CNN
+F 2 "0805" H 3850 1650 60  0001 C CNN
+F 3 "" H 3850 1650 60  0001 C CNN
+F 4 "0.059" H 3850 1650 60  0001 C CNN "Price"
+F 5 "Digikey" H 3850 1650 60  0001 C CNN "Retailer"
+F 6 "311-1358-1-ND" H 3850 1650 60  0001 C CNN "Part_Number"
+	1    3850 1650
+	1    0    0    -1
 $EndComp
 $Comp
@@
 L GND #PWR083
 U 1 1 51EB0A96
-P 4000 2000
-F 0 "#PWR083" H 4000 2000 30  0001 C CNN
-F 1 "GND" H 4000 1930 30  0001 C CNN
-F 2 "" H 4000 2000 60  0001 C CNN
-F 3 "" H 4000 2000 60  0001 C CNN
-	1    4000 2000
+P 3850 1800
+F 0 "#PWR083" H 3850 1800 30  0001 C CNN
+F 1 "GND" H 3850 1730 30  0001 C CNN
+F 2 "" H 3850 1800 60  0001 C CNN
+F 3 "" H 3850 1800 60  0001 C CNN
+	1    3850 1800
 	1    0    0    -1
 $EndComp
@@
 P 3850 3500
 F 0 "R5" V 3930 3500 40  0000 C CNN
-F 1 "330" V 3857 3501 40  0000 C CNN
+F 1 "390" V 3857 3501 40  0000 C CNN
 F 2 "0805" H 3850 3500 60  0001 C CNN
 F 3 "" H 3850 3500 60  0001 C CNN
 F 4 "0.021" V 3850 3500 60  0001 C CNN "Price"
 F 5 "Digikey" V 3850 3500 60  0001 C CNN "Retailer"
-F 6 "RMCF0805JT330RCT-ND" V 3850 3500 60  0001 C CNN "Part_Number"
+F 6 "RMCF0805JT390RCT-ND" V 3850 3500 60  0001 C CNN "Part_Number"
 	1    3850 3500
 	-1   0    0    1
@@
 P 3550 3500
 F 0 "R3" V 3630 3500 40  0000 C CNN
-F 1 "1580" V 3557 3501 40  0000 C CNN
+F 1 "200" V 3557 3501 40  0000 C CNN
 F 2 "0805" H 3550 3500 60  0001 C CNN
 F 3 "" H 3550 3500 60  0001 C CNN
@@
 $EndComp
 $Comp
-L SI1967DH U9
-U 1 1 51EB122D
-P 4650 1650
-F 0 "U9" H 4500 1850 50  0000 C CNN
-F 1 "SI1967DH" H 4650 1450 50  0000 C CNN
-F 2 "6-TSSOP" H 4650 1650 50  0001 C CNN
-F 3 "DOCUMENTATION" H 4650 1650 50  0001 C CNN
-F 4 "0.5" H 4650 1650 60  0001 C CNN "Price"
-F 5 "Digikey" H 4650 1650 60  0001 C CNN "Retailer"
-F 6 "SI1967DH-T1-GE3CT-ND" H 4650 1650 60  0001 C CNN "Part_Number"
-	1    4650 1650
-	1    0    0    -1
-$EndComp
-$Comp
 L GND #PWR091
 U 1 1 51EB154E
@@
 Text Label 4050 1650 0    60   ~ 0
 STAT
-Text Label 5050 1550 0    60   ~ 0
-Dmotor
+Text Label 4050 1550 0    60   ~ 0
+IN1
 Text Label 3250 2650 0    60   ~ 0
-Dmotor
+V24
 Text Label 3000 2100 0    60   ~ 0
 Vmotor
-Text Label 4250 1550 2    60   ~ 0
+Text Label 5300 1550 2    60   ~ 0
 Vmotor
-Text Label 5050 1750 0    60   ~ 0
-Vmotor
-Text Label 5100 1650 0    60   ~ 0
-STAT
-Text Label 4050 1750 0    60   ~ 0
-IN1
 Text Label 4850 2950 0    60   ~ 0
 IN1
@@
 Connection ~ 5200 3050
 Wire Wire Line
-	4000 1950 4000 2000
+	3850 1750 3850 1800
 Wire Wire Line
 	3700 3050 3900 3050
@@
 	5500 3050 5500 3450
 Connection ~ 5500 3050
-Connection ~ 5400 3050
-Wire Wire Line
-	4800 3050 5800 3050
 Wire Wire Line
 	6550 3450 6550 3500
@@
 	3550 3750 3550 3850
 Wire Wire Line
-	4300 1550 4000 1550
+	3850 1550 4300 1550
 Wire Wire Line
 	4300 1650 4000 1650
@@
 	5200 3250 5200 3350
 $Comp
-L GND #PWR094
-U 1 1 51EC4101
-P 5400 3650
-F 0 "#PWR094" H 5400 3650 30  0001 C CNN
-F 1 "GND" H 5400 3580 30  0001 C CNN
-F 2 "" H 5400 3650 60  0001 C CNN
-F 3 "" H 5400 3650 60  0001 C CNN
-	1    5400 3650
-	1    0    0    -1
-$EndComp
-Wire Wire Line
-	5400 3550 5400 3650
+L SI1970DH U9
+U 1 1 51ED81C4
+P 4650 1650
+F 0 "U9" H 4550 1850 50  0000 C CNN
+F 1 "SI1970DH" H 4650 1450 50  0000 C CNN
+F 2 "MODULE" H 4650 1650 50  0001 C CNN
+F 3 "DOCUMENTATION" H 4650 1650 50  0001 C CNN
+	1    4650 1650
+	1    0    0    -1
+$EndComp
+Text HLabel 3250 2650 0    60   Input ~ 0
+V24
+Wire Wire Line
+	4800 3050 5800 3050
 $EndSCHEMATC
