File: Schematics/Vin_and_BackUp.sch (KiCad schematic (older format))
At the start: 15 parts, among them U1 TPS2113A, U2 AP7363-33, U9 SI1970DH

Commit message: Moved the .kicad_pcb file to the board folder. Also did some more routing.
Parts:
- C1, C25, C3, C9: footprint 0805 -> c_0805
- C4: footprint 8.3mmx8.3mm -> c_elec_8x10
- D5: footprint 0805 -> LED-0805
- D6: footprint 0603 -> LED-0603
- R2, R22, R3, R5, R6: footprint 0805 -> SM0805
- U9: footprint MODULE -> sot323-6
Changed lines of the file:
@@
 F 0 "C3" H 3850 1700 30  0000 L CNN
 F 1 "1uF" H 3850 1600 30  0000 L CNN
-F 2 "0805" H 3850 1650 60  0001 C CNN
+F 2 "c_0805" H 3850 1650 60  0001 C CNN
 F 3 "" H 3850 1650 60  0001 C CNN
 F 4 "0.059" H 3850 1650 60  0001 C CNN "Price"
@@
 F 0 "R2" V 3630 2900 40  0000 C CNN
 F 1 "4990" V 3557 2901 40  0000 C CNN
-F 2 "0805" H 3550 2900 60  0001 C CNN
+F 2 "SM0805" H 3550 2900 60  0001 C CNN
 F 3 "" H 3550 2900 60  0001 C CNN
 F 4 "0.029" V 3550 2900 60  0001 C CNN "Price"
@@
 F 0 "D5" H 4150 2550 50  0000 C CNN
 F 1 "LED-G-2" H 4150 2350 50  0000 C CNN
-F 2 "0805" H 4150 2450 60  0001 C CNN
+F 2 "LED-0805" H 4150 2450 60  0001 C CNN
 F 3 "" H 4150 2450 60  0001 C CNN
 F 4 "0.068" H 4150 2450 60  0001 C CNN "Price"
@@
 F 0 "R22" V 6380 3450 40  0000 C CNN
 F 1 "51" V 6307 3451 40  0000 C CNN
-F 2 "0805" H 6300 3450 60  0001 C CNN
+F 2 "SM0805" H 6300 3450 60  0001 C CNN
 F 3 "" H 6300 3450 60  0001 C CNN
 F 4 "0.021" V 6300 3450 60  0001 C CNN "Price"
@@
 F 0 "C4" H 5225 3200 30  0000 L CNN
 F 1 "1mF" H 5225 3075 30  0000 L CNN
-F 2 "8.3mmx8.3mm" H 5200 3150 60  0001 C CNN
+F 2 "c_elec_8x10" H 5200 3150 60  0001 C CNN
 F 3 "" H 5200 3150 60  0001 C CNN
 F 4 "0.81" H 5200 3150 60  0001 C CNN "Price"
@@
 F 0 "D6" H 5800 3550 50  0000 C CNN
 F 1 "LED-B-285" H 5850 3350 50  0000 C CNN
-F 2 "0603" H 5800 3450 60  0001 C CNN
+F 2 "LED-0603" H 5800 3450 60  0001 C CNN
 F 3 "" H 5800 3450 60  0001 C CNN
 F 4 "0.194" H 5800 3450 60  0001 C CNN "Price"
@@
 F 0 "C25" H 5725 4700 30  0000 L CNN
 F 1 "0.1uF" H 5550 4600 30  0000 L CNN
-F 2 "0805" H 5700 4650 60  0001 C CNN
+F 2 "c_0805" H 5700 4650 60  0001 C CNN
 F 3 "" H 5700 4650 60  0001 C CNN
 F 4 "0.01152" H 5700 4650 60  0001 C CNN "Price"
@@
 F 0 "C1" H 3850 4600 30  0000 L CNN
 F 1 "10uF" H 3700 4700 30  0000 L CNN
-F 2 "0805" H 3850 4650 60  0001 C CNN
+F 2 "c_0805" H 3850 4650 60  0001 C CNN
 F 3 "" H 3850 4650 60  0001 C CNN
 F 4 "0.11" V 3850 4650 60  0001 C CNN "Price"
@@
 F 0 "C9" H 5350 4600 30  0000 L CNN
 F 1 "10uF" H 5200 4700 30  0000 L CNN
-F 2 "0805" H 5350 4650 60  0001 C CNN
+F 2 "c_0805" H 5350 4650 60  0001 C CNN
 F 3 "" H 5350 4650 60  0001 C CNN
 F 4 "0.11" V 5350 4650 60  0001 C CNN "Price"
@@
 F 0 "R5" V 3930 3500 40  0000 C CNN
 F 1 "390" V 3857 3501 40  0000 C CNN
-F 2 "0805" H 3850 3500 60  0001 C CNN
+F 2 "SM0805" H 3850 3500 60  0001 C CNN
 F 3 "" H 3850 3500 60  0001 C CNN
 F 4 "0.021" V 3850 3500 60  0001 C CNN "Price"
@@
 F 0 "R3" V 3630 3500 40  0000 C CNN
 F 1 "200" V 3557 3501 40  0000 C CNN
-F 2 "0805" H 3550 3500 60  0001 C CNN
+F 2 "SM0805" H 3550 3500 60  0001 C CNN
 F 3 "" H 3550 3500 60  0001 C CNN
 F 4 "0.029" V 3550 3500 60  0001 C CNN "Price"
@@
 F 0 "R6" V 3730 2150 40  0000 C CNN
 F 1 "200" V 3657 2151 40  0000 C CNN
-F 2 "0805" H 3650 2150 60  0001 C CNN
+F 2 "SM0805" H 3650 2150 60  0001 C CNN
 F 3 "" H 3650 2150 60  0001 C CNN
 F 4 "0.029" V 3650 2150 60  0001 C CNN "Price"
@@
 F 0 "U9" H 4550 1850 50  0000 C CNN
 F 1 "SI1970DH" H 4650 1450 50  0000 C CNN
-F 2 "MODULE" H 4650 1650 50  0001 C CNN
+F 2 "sot323-6" H 4650 1650 50  0001 C CNN
 F 3 "DOCUMENTATION" H 4650 1650 50  0001 C CNN
 	1    4650 1650

Commit message: This commit is to fix the bad push from a bad merger.
Changed lines of the file:
@@
 L GND #PWR084
 U 1 1 51EB0EDC
-P 3000 4350
-F 0 "#PWR084" H 3000 4350 30  0001 C CNN
-F 1 "GND" H 3000 4280 30  0001 C CNN
-F 2 "" H 3000 4350 60  0001 C CNN
-F 3 "" H 3000 4350 60  0001 C CNN
-	1    3000 4350
+P 3950 4450
+F 0 "#PWR084" H 3950 4450 30  0001 C CNN
+F 1 "GND" H 3950 4380 30  0001 C CNN
+F 2 "" H 3950 4450 60  0001 C CNN
+F 3 "" H 3950 4450 60  0001 C CNN
+	1    3950 4450
 	1    0    0    -1
 $EndComp
@@
 L GND #PWR085
 U 1 1 51EB0EE2
-P 3850 4800
-F 0 "#PWR085" H 3850 4800 30  0001 C CNN
-F 1 "GND" H 3850 4730 30  0001 C CNN
-F 2 "" H 3850 4800 60  0001 C CNN
-F 3 "" H 3850 4800 60  0001 C CNN
-	1    3850 4800
+P 3750 4700
+F 0 "#PWR085" H 3750 4700 30  0001 C CNN
+F 1 "GND" H 3750 4630 30  0001 C CNN
+F 2 "" H 3750 4700 60  0001 C CNN
+F 3 "" H 3750 4700 60  0001 C CNN
+	1    3750 4700
 	1    0    0    -1
 $EndComp
@@
 L CSMALL C1
 U 1 1 51EB0F02
-P 3850 4650
-F 0 "C1" H 3850 4600 30  0000 L CNN
-F 1 "10uF" H 3700 4700 30  0000 L CNN
-F 2 "c_0805" H 3850 4650 60  0001 C CNN
-F 3 "" H 3850 4650 60  0001 C CNN
-F 4 "0.11" V 3850 4650 60  0001 C CNN "Price"
-F 5 "Digikey" H 3850 4650 60  0001 C CNN "Retailer"
-F 6 "311-1355-1-ND" H 3850 4650 60  0001 C CNN "Part_Number"
-	1    3850 4650
+P 3750 4550
+F 0 "C1" H 3750 4500 30  0000 L CNN
+F 1 "10uF" H 3600 4600 30  0000 L CNN
+F 2 "c_0805" H 3750 4550 60  0001 C CNN
+F 3 "" H 3750 4550 60  0001 C CNN
+F 4 "0.11" V 3750 4550 60  0001 C CNN "Price"
+F 5 "Digikey" H 3750 4550 60  0001 C CNN "Retailer"
+F 6 "311-1355-1-ND" H 3750 4550 60  0001 C CNN "Part_Number"
+	1    3750 4550
 	-1   0    0    1
 $EndComp
@@
 Text HLabel 2950 2100 0    60   Input ~ 0
 Vmotor
-Text HLabel 3650 4400 0    60   Input ~ 0
+Text HLabel 3550 4300 0    60   Input ~ 0
 Vbatt
 $Comp
@@
 	5700 4750 5700 4800
 Wire Wire Line
-	3850 4750 3850 4800
+	3750 4650 3750 4700
 Wire Wire Line
 	5350 4750 5350 4800
 Wire Wire Line
-	3650 4400 4050 4400
-Wire Wire Line
-	3850 4400 3850 4550
+	3550 4300 4050 4300
+Wire Wire Line
+	3750 4300 3750 4450
 Wire Wire Line
 	5150 4400 5700 4400
@@
 Wire Wire Line
 	5500 3450 5600 3450
-Wire Wire Line
-	3000 4350 3000 4300
-Wire Wire Line
-	3000 4300 4050 4300
-Connection ~ 3850 4400
+Connection ~ 3750 4300
 Wire Wire Line
 	5600 3050 5600 2800
@@
 NoConn ~ 5300 1750
 NoConn ~ 4000 1750
+Wire Wire Line
+	4050 4400 3950 4400
+Wire Wire Line
+	3950 4400 3950 4450
 $EndSCHEMATC

Commit message: More routing stuffs complete.
Connections:
- net labels added: NFET_3, SW_PWR3
- wire segments 45 -> 46
- no-connect marks 3 -> 0
Changed lines of the file:
@@
 L CSMALL C3
 U 1 1 51EB0A40
-P 3850 1650
-F 0 "C3" H 3850 1700 30  0000 L CNN
-F 1 "1uF" H 3850 1600 30  0000 L CNN
-F 2 "c_0805" H 3850 1650 60  0001 C CNN
-F 3 "" H 3850 1650 60  0001 C CNN
-F 4 "0.059" H 3850 1650 60  0001 C CNN "Price"
-F 5 "Digikey" H 3850 1650 60  0001 C CNN "Retailer"
-F 6 "311-1358-1-ND" H 3850 1650 60  0001 C CNN "Part_Number"
-	1    3850 1650
+P 3450 1650
+F 0 "C3" H 3450 1700 30  0000 L CNN
+F 1 "1uF" H 3450 1600 30  0000 L CNN
+F 2 "c_0805" H 3450 1650 60  0001 C CNN
+F 3 "" H 3450 1650 60  0001 C CNN
+F 4 "0.059" H 3450 1650 60  0001 C CNN "Price"
+F 5 "Digikey" H 3450 1650 60  0001 C CNN "Retailer"
+F 6 "311-1358-1-ND" H 3450 1650 60  0001 C CNN "Part_Number"
+	1    3450 1650
 	1    0    0    -1
 $EndComp
@@
 L GND #PWR083
 U 1 1 51EB0A96
-P 3850 1800
-F 0 "#PWR083" H 3850 1800 30  0001 C CNN
-F 1 "GND" H 3850 1730 30  0001 C CNN
-F 2 "" H 3850 1800 60  0001 C CNN
-F 3 "" H 3850 1800 60  0001 C CNN
-	1    3850 1800
+P 3450 1800
+F 0 "#PWR083" H 3450 1800 30  0001 C CNN
+F 1 "GND" H 3450 1730 30  0001 C CNN
+F 2 "" H 3450 1800 60  0001 C CNN
+F 3 "" H 3450 1800 60  0001 C CNN
+	1    3450 1800
 	1    0    0    -1
 $EndComp
@@
 L +3.3V #PWR092
 U 1 1 51EB404B
-P 3650 1850
-F 0 "#PWR092" H 3650 1810 30  0001 C CNN
-F 1 "+3.3V" H 3650 1960 30  0000 C CNN
-F 2 "" H 3650 1850 60  0001 C CNN
-F 3 "" H 3650 1850 60  0001 C CNN
-	1    3650 1850
+P 3650 1900
+F 0 "#PWR092" H 3650 1860 30  0001 C CNN
+F 1 "+3.3V" H 3650 2010 30  0000 C CNN
+F 2 "" H 3650 1900 60  0001 C CNN
+F 3 "" H 3650 1900 60  0001 C CNN
+	1    3650 1900
 	1    0    0    -1
 $EndComp
@@
 Connection ~ 5200 3050
 Wire Wire Line
-	3850 1750 3850 1800
+	3450 1750 3450 1800
 Wire Wire Line
 	3700 3050 3900 3050
@@
 	3550 3750 3550 3850
 Wire Wire Line
-	3850 1550 4300 1550
+	3450 1550 4300 1550
 Wire Wire Line
 	4300 1650 4000 1650
-Wire Wire Line
-	4300 1750 4000 1750
 Wire Wire Line
 	5000 1550 5300 1550
@@
 Connection ~ 5600 3050
 Wire Wire Line
-	3650 1900 3650 1850
+	3650 1900 3650 1900
 Connection ~ 3650 2450
 $Comp
@@
 Wire Wire Line
 	4800 3050 5800 3050
-NoConn ~ 5300 1650
-NoConn ~ 5300 1750
-NoConn ~ 4000 1750
 Wire Wire Line
 	4050 4400 3950 4400
 Wire Wire Line
 	3950 4400 3950 4450
+Text Label 4300 1750 2    60   ~ 0
+SW_PWR3
+$Comp
+L GND #PWR?
+U 1 1 51F2D6E1
+P 5300 1800
+F 0 "#PWR?" H 5300 1800 30  0001 C CNN
+F 1 "GND" H 5300 1730 30  0001 C CNN
+F 2 "" H 5300 1800 60  0001 C CNN
+F 3 "" H 5300 1800 60  0001 C CNN
+	1    5300 1800
+	1    0    0    -1
+$EndComp
+Wire Wire Line
+	4300 1750 4000 1750
+Wire Wire Line
+	5300 1750 5300 1800
+Text Label 5000 1650 0    60   ~ 0
+NFET_3
+Text HLabel 5300 1650 2    60   Input ~ 0
+NFET_3
+Text HLabel 4000 1750 0    60   Input ~ 0
+SW_PWR3
 $EndSCHEMATC

Commit message: Started making changes to the Sensor Board for v.2
Parts:
- removed C3: 1uF, c_0805, symbol CSMALL
- removed C4: 1mF, c_elec_8x10, symbol CPSMALL
- removed R2: 4990, SM0805, symbol R
- removed R3: 200, SM0805, symbol R
- removed R5: 390, SM0805, symbol R
- removed U1: TPS2113A, 8-TSSOP, symbol TPS2113A
Connections:
- net labels added: XBEE_NFET, XBEE_PWR
- net labels removed: IN1, NFET_3, STAT, SW_PWR3, V24, VLDO, Vmotor
- wire segments 46 -> 21
Other:
- note removed: "1%"
- moved on the sheet: R22, R6
