File: Schematics/Vin_and_BackUp.sch (KiCad schematic (older format))
At the start: 9 parts, among them U2 AP7363-33, U9 SI1970DH

Commit message: Almost finished with V2.0 of the sensor board. Need to add one more trace... hopefully.
Parts:
- removed D6: LED-B-285, LED-0603, symbol LED
- removed R22: 51, SM0805, symbol R
Connections:
- net labels added: NFET_3, PWR_SW3, V33
- wire segments 21 -> 23
Other:
- note removed: "BLUE"
- moved on the sheet: R6
Changed lines of the file:
@@
 LIBS:microclasp_hdrx3
 LIBS:pinhd-2x23
+LIBS:ld29150dt50r
+LIBS:ncp59151ds50r4g
 LIBS:Sensor_Board-cache
 EELAYER 27 0
@@
 $Descr A4 11693 8268
 encoding utf-8
-Sheet 3 3
+Sheet 3 4
 Title ""
-Date "31 dec 2013"
+Date "8 jan 2014"
 Rev ""
 Comp ""
@@
 L LED D5
 U 1 1 51EB0A64
-P 3900 5550
-F 0 "D5" H 3900 5650 50  0000 C CNN
-F 1 "LED-G-2" H 3900 5450 50  0000 C CNN
-F 2 "LED-0805" H 3900 5550 60  0001 C CNN
-F 3 "" H 3900 5550 60  0001 C CNN
-F 4 "0.068" H 3900 5550 60  0001 C CNN "Price"
-F 5 "Digikey" H 3900 5550 60  0001 C CNN "Retailer"
-F 6 "475-1410-1-ND" H 3900 5550 60  0001 C CNN "Part_Number"
-	1    3900 5550
-	1    0    0    -1
-$EndComp
-$Comp
-L GND #PWR086
-U 1 1 51EB0A6A
-P 4950 3500
-F 0 "#PWR086" H 4950 3500 30  0001 C CNN
-F 1 "GND" H 4950 3430 30  0001 C CNN
-F 2 "" H 4950 3500 60  0001 C CNN
-F 3 "" H 4950 3500 60  0001 C CNN
-	1    4950 3500
-	1    0    0    -1
-$EndComp
-$Comp
-L R R22
-U 1 1 51EB0A73
-P 4700 3450
-F 0 "R22" V 4780 3450 40  0000 C CNN
-F 1 "51" V 4707 3451 40  0000 C CNN
-F 2 "SM0805" H 4700 3450 60  0001 C CNN
-F 3 "" H 4700 3450 60  0001 C CNN
-F 4 "0.021" V 4700 3450 60  0001 C CNN "Price"
-F 5 "Digikey" V 4700 3450 60  0001 C CNN "Retailer"
-F 6 "RMCF0805JT51R0CT-ND" V 4700 3450 60  0001 C CNN "Part_Number"
-	1    4700 3450
-	0    -1   -1   0
-$EndComp
-Text Notes 4150 3300 0    60   ~ 0
-BLUE
-$Comp
-L LED D6
-U 1 1 51EB0A8C
-P 4200 3450
-F 0 "D6" H 4200 3550 50  0000 C CNN
-F 1 "LED-B-285" H 4250 3350 50  0000 C CNN
-F 2 "LED-0603" H 4200 3450 60  0001 C CNN
-F 3 "" H 4200 3450 60  0001 C CNN
-F 4 "0.194" H 4200 3450 60  0001 C CNN "Price"
-F 5 "Digikey" H 4200 3450 60  0001 C CNN "Retailer"
-F 6 "475-2815-1-ND" H 4200 3450 60  0001 C CNN "Part_Number"
-	1    4200 3450
-	1    0    0    -1
-$EndComp
-Text Notes 3750 5800 0    60   ~ 0
+P 4800 5750
+F 0 "D5" H 4800 5850 50  0000 C CNN
+F 1 "LED-G-2" H 4800 5650 50  0000 C CNN
+F 2 "LED-0805" H 4800 5750 60  0001 C CNN
+F 3 "" H 4800 5750 60  0001 C CNN
+F 4 "0.068" H 4800 5750 60  0001 C CNN "Price"
+F 5 "Digikey" H 4800 5750 60  0001 C CNN "Retailer"
+F 6 "475-1410-1-ND" H 4800 5750 60  0001 C CNN "Part_Number"
+	1    4800 5750
+	1    0    0    -1
+$EndComp
+Text Notes 4650 6000 0    60   ~ 0
 GREEN
 $Comp
@@
 $EndComp
 $Comp
-L GND #PWR088
+L GND #PWR0102
 U 1 1 51EB0EDC
 P 3950 4450
-F 0 "#PWR088" H 3950 4450 30  0001 C CNN
+F 0 "#PWR0102" H 3950 4450 30  0001 C CNN
 F 1 "GND" H 3950 4380 30  0001 C CNN
 F 2 "" H 3950 4450 60  0001 C CNN
@@
 $EndComp
 $Comp
-L GND #PWR089
+L GND #PWR0103
 U 1 1 51EB0EE2
 P 3750 4700
-F 0 "#PWR089" H 3750 4700 30  0001 C CNN
+F 0 "#PWR0103" H 3750 4700 30  0001 C CNN
 F 1 "GND" H 3750 4630 30  0001 C CNN
 F 2 "" H 3750 4700 60  0001 C CNN
@@
 $EndComp
 $Comp
-L GND #PWR090
+L GND #PWR0104
 U 1 1 51EB0EEA
 P 5350 4800
-F 0 "#PWR090" H 5350 4800 30  0001 C CNN
+F 0 "#PWR0104" H 5350 4800 30  0001 C CNN
 F 1 "GND" H 5350 4730 30  0001 C CNN
 F 2 "" H 5350 4800 60  0001 C CNN
@@
 $EndComp
 $Comp
-L GND #PWR091
+L GND #PWR0105
 U 1 1 51EB0EF0
 P 5700 4800
-F 0 "#PWR091" H 5700 4800 30  0001 C CNN
+F 0 "#PWR0105" H 5700 4800 30  0001 C CNN
 F 1 "GND" H 5700 4730 30  0001 C CNN
 F 2 "" H 5700 4800 60  0001 C CNN
@@
 Vbatt
 $Comp
-L GND #PWR095
+L GND #PWR0106
 U 1 1 51EB154E
-P 4200 5600
-F 0 "#PWR095" H 4200 5600 30  0001 C CNN
-F 1 "GND" H 4200 5530 30  0001 C CNN
-F 2 "" H 4200 5600 60  0001 C CNN
-F 3 "" H 4200 5600 60  0001 C CNN
-	1    4200 5600
-	1    0    0    -1
-$EndComp
-Wire Wire Line
-	4400 3450 4450 3450
-Wire Wire Line
-	4950 3450 4950 3500
+P 5100 5800
+F 0 "#PWR0106" H 5100 5800 30  0001 C CNN
+F 1 "GND" H 5100 5730 30  0001 C CNN
+F 2 "" H 5100 5800 60  0001 C CNN
+F 3 "" H 5100 5800 60  0001 C CNN
+	1    5100 5800
+	1    0    0    -1
+$EndComp
 Wire Wire Line
 	5350 4550 5350 4400
@@
 Connection ~ 5350 4400
 Wire Wire Line
-	5000 1650 5300 1650
-Wire Wire Line
-	5000 1750 5300 1750
-Wire Wire Line
-	4200 5550 4200 5600
-Wire Wire Line
-	3900 3450 4000 3450
+	5150 3650 5450 3650
+Wire Wire Line
+	5100 5750 5100 5800
 Connection ~ 3750 4300
 Wire Wire Line
-	4100 5550 4200 5550
+	5000 5750 5100 5750
 $Comp
 L SI1970DH U9
 U 1 1 51ED81C4
-P 4650 1650
-F 0 "U9" H 4550 1850 50  0000 C CNN
-F 1 "SI1970DH" H 4650 1450 50  0000 C CNN
-F 2 "sot323-6" H 4650 1650 50  0001 C CNN
-F 3 "DOCUMENTATION" H 4650 1650 50  0001 C CNN
-	1    4650 1650
+P 4800 3650
+F 0 "U9" H 4700 3850 50  0000 C CNN
+F 1 "SI1970DH" H 4800 3450 50  0000 C CNN
+F 2 "sot323-6" H 4800 3650 50  0001 C CNN
+F 3 "DOCUMENTATION" H 4800 3650 50  0001 C CNN
+	1    4800 3650
 	1    0    0    -1
 $EndComp
@@
 Wire Wire Line
 	3950 4400 3950 4450
-Wire Wire Line
-	3800 1750 4300 1750
-Text HLabel 5300 1750 2    60   Input ~ 0
+Text HLabel 4100 3750 0    60   Output ~ 0
 XBEE_PWR
-$Comp
-L +3.3V #PWR?
-U 1 1 52C23358
-P 3800 1750
-F 0 "#PWR?" H 3800 1710 30  0001 C CNN
-F 1 "+3.3V" H 3800 1860 30  0000 C CNN
-F 2 "" H 3800 1750 60  0000 C CNN
-F 3 "" H 3800 1750 60  0000 C CNN
-	1    3800 1750
-	1    0    0    -1
-$EndComp
-Text HLabel 5300 1650 2    60   Input ~ 0
+Text HLabel 5450 3650 2    60   Input ~ 0
 XBEE_NFET
 $Comp
 L R R6
 U 1 1 51EB4833
-P 3400 5250
-F 0 "R6" V 3480 5250 40  0000 C CNN
-F 1 "200" V 3407 5251 40  0000 C CNN
-F 2 "SM0805" H 3400 5250 60  0001 C CNN
-F 3 "" H 3400 5250 60  0001 C CNN
-F 4 "0.029" V 3400 5250 60  0001 C CNN "Price"
-F 5 "Digikey" V 3400 5250 60  0001 C CNN "Retailer"
-F 6 "RMCF0805JT200RCT-ND" V 3400 5250 60  0001 C CNN "Part_Number"
-	1    3400 5250
+P 4300 5450
+F 0 "R6" V 4380 5450 40  0000 C CNN
+F 1 "200" V 4307 5451 40  0000 C CNN
+F 2 "SM0805" H 4300 5450 60  0001 C CNN
+F 3 "" H 4300 5450 60  0001 C CNN
+F 4 "0.029" V 4300 5450 60  0001 C CNN "Price"
+F 5 "Digikey" V 4300 5450 60  0001 C CNN "Retailer"
+F 6 "RMCF0805JT200RCT-ND" V 4300 5450 60  0001 C CNN "Part_Number"
+	1    4300 5450
 	-1   0    0    1
 $EndComp
-Connection ~ 3400 5550
-Wire Wire Line
-	3400 5000 3400 5000
-Wire Wire Line
-	3400 5550 3700 5550
-$Comp
-L +3.3V #PWR096
+Connection ~ 4300 5750
+Wire Wire Line
+	4300 5200 4300 5200
+Wire Wire Line
+	4300 5750 4600 5750
+$Comp
+L +3.3V #PWR0107
 U 1 1 51EB404B
-P 3400 5000
-F 0 "#PWR096" H 3400 4960 30  0001 C CNN
-F 1 "+3.3V" H 3400 5110 30  0000 C CNN
-F 2 "" H 3400 5000 60  0001 C CNN
-F 3 "" H 3400 5000 60  0001 C CNN
-	1    3400 5000
-	1    0    0    -1
-$EndComp
-Wire Wire Line
-	3400 5500 3400 5550
-Text HLabel 5850 4400 2    60   Input ~ 0
-Vin
+P 4300 5200
+F 0 "#PWR0107" H 4300 5160 30  0001 C CNN
+F 1 "+3.3V" H 4300 5310 30  0000 C CNN
+F 2 "" H 4300 5200 60  0001 C CNN
+F 3 "" H 4300 5200 60  0001 C CNN
+	1    4300 5200
+	1    0    0    -1
+$EndComp
+Wire Wire Line
+	4300 5700 4300 5750
+Text HLabel 5850 4400 2    60   Output ~ 0
+V33
 Connection ~ 5700 4400
 Text Label 5450 4400 0    60   ~ 0
 Vin
+Wire Wire Line
+	4450 3750 4100 3750
+$Comp
+L GND #PWR0108
+U 1 1 52C71A9C
+P 5300 3850
+F 0 "#PWR0108" H 5300 3850 30  0001 C CNN
+F 1 "GND" H 5300 3780 30  0001 C CNN
+F 2 "" H 5300 3850 60  0001 C CNN
+F 3 "" H 5300 3850 60  0001 C CNN
+	1    5300 3850
+	1    0    0    -1
+$EndComp
+Wire Wire Line
+	5150 3750 5300 3750
+Wire Wire Line
+	5300 3750 5300 3850
+Wire Wire Line
+	5150 3550 5450 3550
+Wire Wire Line
+	3500 3550 4450 3550
+Wire Wire Line
+	4450 3650 4100 3650
+$Comp
+L GND #PWR0109
+U 1 1 52C87942
+P 3500 3600
+F 0 "#PWR0109" H 3500 3600 30  0001 C CNN
+F 1 "GND" H 3500 3530 30  0001 C CNN
+F 2 "" H 3500 3600 60  0001 C CNN
+F 3 "" H 3500 3600 60  0001 C CNN
+	1    3500 3600
+	1    0    0    -1
+$EndComp
+Text HLabel 5450 3550 2    60   Output ~ 0
+PWR_SW3
+Wire Wire Line
+	3500 3550 3500 3600
+Text HLabel 4100 3650 0    60   Input ~ 0
+NFET_3
 $EndSCHEMATC
