File: Schematics/BBB_Pins.sch (KiCad schematic (older format))
At the start: 9 parts, among them U1 NCP59151DS50R4G, U3 SN65HVD232

Commit message: Minor Changes to original Sensor Board design
Parts:
- C3, C4: symbol C -> C-RESCUE-Sensor_Board
- D7: symbol LED -> LED-RESCUE-Sensor_Board
- R35, R36: symbol R -> R-RESCUE-Sensor_Board
Changed lines of the file:
@@
 EESchema Schematic File Version 2
+LIBS:Sensor_Board-rescue
 LIBS:power
 LIBS:device
@@
 LIBS:memory
 LIBS:xilinx
-LIBS:special
 LIBS:microcontrollers
 LIBS:dsp
@@
 LIBS:TPS2113A
 LIBS:Sensor_Board-cache
-EELAYER 24 0
+EELAYER 25 0
 EELAYER END
 $Descr A4 11693 8268
@@
 Vin
 $Comp
-L GND #PWR0109
+L GND-RESCUE-Sensor_Board #PWR0109
 U 1 1 52C60290
 P 1450 1600
-F 0 "#PWR0109" H 1450 1600 30  0001 C CNN
+AR Path="/52C60290" Ref="#PWR0109"  Part="1"
+AR Path="/52C5CC47/52C60290" Ref="#PWR0110"  Part="1"
+F 0 "#PWR0110" H 1450 1600 30  0001 C CNN
 F 1 "GND" H 1450 1530 30  0001 C CNN
 F 2 "" H 1450 1600 60  0001 C CNN
@@
 $EndComp
 $Comp
-L R R35
+L R-RESCUE-Sensor_Board R35
 U 1 1 52C60299
 P 1600 2200
+AR Path="/52C60299" Ref="R35"  Part="1"
+AR Path="/52C5CC47/52C60299" Ref="R35"  Part="1"
 F 0 "R35" V 1680 2200 40  0000 C CNN
 F 1 "200" V 1607 2201 40  0000 C CNN
@@
 BLUE
 $Comp
-L LED D7
+L LED-RESCUE-Sensor_Board D7
 U 1 1 52C602A3
 P 1100 2200
+AR Path="/52C602A3" Ref="D7"  Part="1"
+AR Path="/52C5CC47/52C602A3" Ref="D7"  Part="1"
 F 0 "D7" H 1100 2300 50  0000 C CNN
 F 1 "LED-B-285" H 1150 2100 50  0000 C CNN
@@
 	800  2200 900  2200
 $Comp
-L GND #PWR0110
+L GND-RESCUE-Sensor_Board #PWR0110
 U 1 1 52C602CD
 P 2650 1750
-F 0 "#PWR0110" H 2650 1750 30  0001 C CNN
+AR Path="/52C602CD" Ref="#PWR0110"  Part="1"
+AR Path="/52C5CC47/52C602CD" Ref="#PWR0111"  Part="1"
+F 0 "#PWR0111" H 2650 1750 30  0001 C CNN
 F 1 "GND" H 2650 1680 30  0001 C CNN
 F 2 "" H 2650 1750 60  0000 C CNN
@@
 V5
 $Comp
-L +5V #PWR0111
+L +5V #PWR0112
 U 1 1 52C602EE
 P 800 2100
-F 0 "#PWR0111" H 800 2190 20  0001 C CNN
+F 0 "#PWR0112" H 800 2190 20  0001 C CNN
 F 1 "+5V" H 800 2190 30  0000 C CNN
 F 2 "" H 800 2100 60  0000 C CNN
@@
 5V_FLG
 $Comp
-L PWR_FLAG #FLG0112
+L PWR_FLAG #FLG0113
 U 1 1 52C7258E
 P 5150 750
-F 0 "#FLG0112" H 5150 845 30  0001 C CNN
+F 0 "#FLG0113" H 5150 845 30  0001 C CNN
 F 1 "PWR_FLAG" H 5150 930 30  0000 C CNN
 F 2 "" H 5150 750 60  0000 C CNN
@@
 $EndComp
 $Comp
-L +5V #PWR0113
+L +5V #PWR0114
 U 1 1 52C72768
 P 5150 900
-F 0 "#PWR0113" H 5150 990 20  0001 C CNN
+F 0 "#PWR0114" H 5150 990 20  0001 C CNN
 F 1 "+5V" H 5150 990 30  0000 C CNN
 F 2 "" H 5150 900 60  0000 C CNN
@@
 	5150 750  5150 900
 $Comp
-L GND #PWR0114
+L GND-RESCUE-Sensor_Board #PWR0114
 U 1 1 52C74550
 P 4150 2350
-F 0 "#PWR0114" H 4150 2350 30  0001 C CNN
+AR Path="/52C74550" Ref="#PWR0114"  Part="1"
+AR Path="/52C5CC47/52C74550" Ref="#PWR0115"  Part="1"
+F 0 "#PWR0115" H 4150 2350 30  0001 C CNN
 F 1 "GND" H 4150 2280 30  0001 C CNN
 F 2 "" H 4150 2350 60  0000 C CNN
@@
 NoConn ~ 5050 2400
 $Comp
-L +5V #PWR0115
+L +5V #PWR0116
 U 1 1 52C745EE
 P 3800 1150
-F 0 "#PWR0115" H 3800 1240 20  0001 C CNN
+F 0 "#PWR0116" H 3800 1240 20  0001 C CNN
 F 1 "+5V" H 3800 1240 30  0000 C CNN
 F 2 "" H 3800 1150 60  0000 C CNN
@@
 $EndComp
 $Comp
-L +5V #PWR0116
+L +5V #PWR0117
 U 1 1 52C745F4
 P 4300 2450
-F 0 "#PWR0116" H 4300 2540 20  0001 C CNN
+F 0 "#PWR0117" H 4300 2540 20  0001 C CNN
 F 1 "+5V" H 4300 2540 30  0000 C CNN
 F 2 "" H 4300 2450 60  0000 C CNN
@@
 BBB_CAN_RX
 $Comp
-L GND #PWR0117
+L GND-RESCUE-Sensor_Board #PWR0117
 U 1 1 52C74886
 P 1650 3550
-F 0 "#PWR0117" H 1650 3550 30  0001 C CNN
+AR Path="/52C74886" Ref="#PWR0117"  Part="1"
+AR Path="/52C5CC47/52C74886" Ref="#PWR0118"  Part="1"
+F 0 "#PWR0118" H 1650 3550 30  0001 C CNN
 F 1 "GND" H 1650 3480 30  0001 C CNN
 F 2 "" H 1650 3550 60  0001 C CNN
@@
 $EndComp
 $Comp
-L +3.3V #PWR0118
+L +3.3V-RESCUE-Sensor_Board #PWR0118
 U 1 1 52C7489E
 P 1800 3600
-F 0 "#PWR0118" H 1800 3560 30  0001 C CNN
+AR Path="/52C7489E" Ref="#PWR0118"  Part="1"
+AR Path="/52C5CC47/52C7489E" Ref="#PWR0119"  Part="1"
+F 0 "#PWR0119" H 1800 3560 30  0001 C CNN
 F 1 "+3.3V" H 1800 3710 30  0000 C CNN
 F 2 "" H 1800 3600 60  0001 C CNN
@@
 	2000 1350 2100 1350
 $Comp
-L C C3
+L C-RESCUE-Sensor_Board C3
 U 1 1 52CC5F13
 P 1450 1350
+AR Path="/52CC5F13" Ref="C3"  Part="1"
+AR Path="/52C5CC47/52CC5F13" Ref="C3"  Part="1"
 F 0 "C3" H 1450 1450 40  0000 L CNN
 F 1 "1uF" H 1456 1265 40  0000 L CNN
@@
 	1450 1550 1450 1600
 $Comp
-L R R36
+L R-RESCUE-Sensor_Board R36
 U 1 1 52CC5FF4
 P 3350 1400
+AR Path="/52CC5FF4" Ref="R36"  Part="1"
+AR Path="/52C5CC47/52CC5FF4" Ref="R36"  Part="1"
 F 0 "R36" V 3430 1400 40  0000 C CNN
 F 1 "100k" V 3357 1401 40  0000 C CNN
@@
 Connection ~ 1450 1150
 $Comp
-L C C4
+L C-RESCUE-Sensor_Board C4
 U 1 1 52CC60AF
 P 3600 1350
+AR Path="/52CC60AF" Ref="C4"  Part="1"
+AR Path="/52C5CC47/52CC60AF" Ref="C4"  Part="1"
 F 0 "C4" H 3600 1450 40  0000 L CNN
 F 1 "47uF" H 3606 1265 40  0000 L CNN
@@
 $EndComp
 $Comp
-L GND #PWR0119
+L GND-RESCUE-Sensor_Board #PWR0119
 U 1 1 52CC60BC
 P 1850 2250
-F 0 "#PWR0119" H 1850 2250 30  0001 C CNN
+AR Path="/52CC60BC" Ref="#PWR0119"  Part="1"
+AR Path="/52C5CC47/52CC60BC" Ref="#PWR0120"  Part="1"
+F 0 "#PWR0120" H 1850 2250 30  0001 C CNN
 F 1 "GND" H 1850 2180 30  0001 C CNN
 F 2 "" H 1850 2250 60  0001 C CNN
@@
 $EndComp
 $Comp
-L GND #PWR0120
+L GND-RESCUE-Sensor_Board #PWR0120
 U 1 1 52CC60C2
 P 3600 1550
-F 0 "#PWR0120" H 3600 1550 30  0001 C CNN
+AR Path="/52CC60C2" Ref="#PWR0120"  Part="1"
+AR Path="/52C5CC47/52CC60C2" Ref="#PWR0121"  Part="1"
+F 0 "#PWR0121" H 3600 1550 30  0001 C CNN
 F 1 "GND" H 3600 1480 30  0001 C CNN
 F 2 "" H 3600 1550 60  0001 C CNN
